Commit message: Add Tigra Description

File: tigra_description/urdf/robot.urdf.xacro (robot description, xacro)
@@ -88,4 +88,5 @@
 </xacro:macro>
 <!-- zawarka solution -->
+<!-- speed -->
 <xacro:macro name="speed_wheel" params="name base_name xyz ">
     <xacro:wheels name="wheel_${name}" />
@@ -94,27 +95,15 @@
     </link>
     <joint name="${name}_spring_joint" type="prismatic">
-    <limit lower="-0.000000001" upper="0.000000001" effort="0" velocity="0"/>
+    <limit lower="-0.00001" upper="0.00001" effort="0" velocity="0"/>
       <parent link="${base_name}"/>
       <child link="spring1_${name}"/>
-      	<axis>
-      		<dynamics>
-      			<spring_stiffness>420000</spring_stiffness>
-      			<spring_reference>1</spring_reference>
-     			<damping>100000000</damping>
-      			<friction>100</friction>
-    		</dynamics>
-    		<use_parent_model_frame>0</use_parent_model_frame>
-  		</axis>
-  		<physics>
-    		<ode>
-      			<implicit_spring_damper>1</implicit_spring_damper>
-      			<cfm_damping>1</cfm_damping>
-      				<limit>
-        				<cfm>0</cfm>
-        				<erp>0.2</erp>
-      				</limit>
-    		</ode>
-  		</physics>
+	  <dynamics damping="0.0" friction="0.0"/>
+	  <axis xyz="0 0 1"/>
     </joint>
+  <gazebo reference="${name}_spring_joint">
+    <implicitSpringDamper>true</implicitSpringDamper>
+    <springStiffness>4200</springStiffness>
+    <springReference>0.2</springReference>
+  </gazebo>
     <joint name="${name}_speed_joint" type="continuous">
       <parent link="spring1_${name}"/>
@@ -125,4 +114,5 @@
     </joint>
 </xacro:macro>
+<!-- steer -->
 <xacro:macro name="steer_wheel" params="name base_name xyz">
     <xacro:wheels name="wheel_${name}" />
@@ -134,5 +124,5 @@
     </link>
     <joint name="${name}_spring_joint" type="prismatic">
-    <limit lower="-0.000000001" upper="0.000000001" effort="0" velocity="0"/>
+    <limit lower="-0.01" upper="0.01" effort="0" velocity="0"/>
       <parent link="${base_name}"/>
       <child link="spring2_${name}"/>
@@ -174,12 +164,13 @@
     </joint>
 </xacro:macro>
-	<xacro:steer_wheel name="joint_right_wheel_1" base_name="base_link" xyz="0.5 -0.375 -0.3" />
-	<xacro:steer_wheel name="joint_left_wheel_1" base_name="base_link" xyz="0.5 0.375 -0.3" />
-	<xacro:speed_wheel name="joint_right_wheel_2" base_name="base_link" xyz="-0.5 -0.375 -0.3" />
-	<xacro:speed_wheel name="joint_left_wheel_2" base_name="base_link" xyz="-0.55 0.375 -0.3" />
+<!-- steer_wheel -->
+	<xacro:speed_wheel name="joint_right_wheel_1" base_name="base_link" xyz="0.5 -0.375 -0.35" />
+	<xacro:speed_wheel name="joint_left_wheel_1" base_name="base_link" xyz="0.5 0.375 -0.35" />
+<!-- speed_wheel -->
+	<xacro:speed_wheel name="joint_right_wheel_2" base_name="base_link" xyz="-0.5 -0.375 -0.35" />
+	<xacro:speed_wheel name="joint_left_wheel_2" base_name="base_link" xyz="-0.5 0.375 -0.35" />
 <!--<gazebo>
     <plugin name="ModelPlugin" filename="librobot_gazebo.so" >
       <robotName>tigra</robotName>
-      <wheelbase>base_link</wheelbase>
       <_joint>joint_right_wheel_2_speed_joint</_joint>
     </plugin>

Commit message: Weight monitoring

File: tigra_description/urdf/robot.urdf.xacro (robot description, xacro)
@@ -4,12 +4,10 @@
 <xacro:property name="width" value="0.75" />
 <xacro:property name="heigth" value="0.6" />
-<xacro:property name="mass" value="420" />
+<xacro:property name="mass" value="0.42" />
 <xacro:property name="wheel_width" value="0.25" />
 <xacro:property name="wheel_radius" value="0.25" />
-<xacro:property name="wheel_mass" value="20" />
+<xacro:property name="wheel_mass" value="0.02" />
 <xacro:property name="wheel_turn_limit" value="${pi/4}"/>
-<xacro:property name="wheelbase" value="1.24" />
-<xacro:property name="trackbase" value="1.00" />
-<xacro:property name="base_center" value="${length/2}" />
+<xacro:property name="springStiffness" value="105" />
 <!-- inertia -->
 <xacro:macro name="null_inertial">
@@ -94,6 +92,11 @@
       <xacro:null_inertial/>
     </link>
+    <gazebo reference="${name}_spring_joint">
+    	<implicitSpringDamper>true</implicitSpringDamper>
+    	<springStiffness>${springStiffness}</springStiffness>
+    	<springReference>0</springReference>
+    </gazebo>
     <joint name="${name}_spring_joint" type="prismatic">
-    <limit lower="-0.00001" upper="0.00001" effort="0" velocity="0"/>
+    <limit lower="-0.05" upper="0.05" effort="0" velocity="0"/>
       <parent link="${base_name}"/>
       <child link="spring1_${name}"/>
@@ -101,9 +104,4 @@
 	  <axis xyz="0 0 1"/>
     </joint>
-  <gazebo reference="${name}_spring_joint">
-    <implicitSpringDamper>true</implicitSpringDamper>
-    <springStiffness>4200</springStiffness>
-    <springReference>0.2</springReference>
-  </gazebo>
     <joint name="${name}_speed_joint" type="continuous">
       <parent link="spring1_${name}"/>
@@ -123,27 +121,15 @@
       <xacro:null_inertial/>
     </link>
+    <gazebo reference="${name}_spring_joint">
+    	<implicitSpringDamper>true</implicitSpringDamper>
+    	<springStiffness>${springStiffness}</springStiffness>
+    	<springReference>0</springReference>
+    </gazebo>
     <joint name="${name}_spring_joint" type="prismatic">
-    <limit lower="-0.01" upper="0.01" effort="0" velocity="0"/>
+    <limit lower="-0.05" upper="0.05" effort="0" velocity="0"/>
       <parent link="${base_name}"/>
       <child link="spring2_${name}"/>
-      	<axis>
-      		<dynamics>
-      			<spring_stiffness>420000</spring_stiffness>
-      			<spring_reference>1</spring_reference>
-     			<damping>100000000</damping>
-      			<friction>100</friction>
-    		</dynamics>
-    		<use_parent_model_frame>0</use_parent_model_frame>
-  		</axis>
-  		<physics>
-    		<ode>
-      			<implicit_spring_damper>1</implicit_spring_damper>
-      			<cfm_damping>1</cfm_damping>
-      				<limit>
-        				<cfm>0</cfm>
-        				<erp>0.2</erp>
-      				</limit>
-    		</ode>
-  		</physics>
+	  <dynamics damping="0.0" friction="0.0"/>
+	  <axis xyz="0 0 1"/>
     </joint>
     <joint name="${name}_steer_joint" type="revolute">
@@ -165,14 +151,8 @@
 </xacro:macro>
 <!-- steer_wheel -->
-	<xacro:speed_wheel name="joint_right_wheel_1" base_name="base_link" xyz="0.5 -0.375 -0.35" />
-	<xacro:speed_wheel name="joint_left_wheel_1" base_name="base_link" xyz="0.5 0.375 -0.35" />
+	<xacro:steer_wheel name="joint_right_wheel_1" base_name="base_link" xyz="0.5 -0.375 -0.35" />
+	<xacro:steer_wheel name="joint_left_wheel_1" base_name="base_link" xyz="0.5 0.375 -0.35" />
 <!-- speed_wheel -->
 	<xacro:speed_wheel name="joint_right_wheel_2" base_name="base_link" xyz="-0.5 -0.375 -0.35" />
 	<xacro:speed_wheel name="joint_left_wheel_2" base_name="base_link" xyz="-0.5 0.375 -0.35" />
-<!--<gazebo>
-    <plugin name="ModelPlugin" filename="librobot_gazebo.so" >
-      <robotName>tigra</robotName>
-      <_joint>joint_right_wheel_2_speed_joint</_joint>
-    </plugin>
-</gazebo> -->
 </robot>

Commit message: Revolute problem

File: tigra_description/urdf/robot.urdf.xacro (robot description, xacro)
@@ -4,8 +4,8 @@
 <xacro:property name="width" value="0.75" />
 <xacro:property name="heigth" value="0.6" />
-<xacro:property name="mass" value="0.42" />
+<xacro:property name="mass" value="420" />
 <xacro:property name="wheel_width" value="0.25" />
 <xacro:property name="wheel_radius" value="0.25" />
-<xacro:property name="wheel_mass" value="0.02" />
+<xacro:property name="wheel_mass" value="20" />
 <xacro:property name="wheel_turn_limit" value="${pi/4}"/>
 <xacro:property name="springStiffness" value="105" />
@@ -89,4 +89,5 @@
 <xacro:macro name="speed_wheel" params="name base_name xyz ">
     <xacro:wheels name="wheel_${name}" />
+<!--
     <link name="spring1_${name}">
       <xacro:null_inertial/>
@@ -104,6 +105,8 @@
 	  <axis xyz="0 0 1"/>
     </joint>
+-->
     <joint name="${name}_speed_joint" type="continuous">
-      <parent link="spring1_${name}"/>
+<!--      <parent link="spring1_${name}"/> -->
+      <parent link="${base_name}"/>
       <child link="wheel_${name}"/>
       <origin xyz="${xyz}" rpy="${pi/2} 0 0"/>
@@ -115,10 +118,13 @@
 <xacro:macro name="steer_wheel" params="name base_name xyz">
     <xacro:wheels name="wheel_${name}" />
+<!--
     <link name="spring2_${name}">
       <xacro:null_inertial/>
     </link>
+-->
      <link name="steer_${name}">
       <xacro:null_inertial/>
     </link>
+<!--
     <gazebo reference="${name}_spring_joint">
     	<implicitSpringDamper>true</implicitSpringDamper>
@@ -133,9 +139,11 @@
 	  <axis xyz="0 0 1"/>
     </joint>
+-->
     <joint name="${name}_steer_joint" type="revolute">
       <limit lower="${-wheel_turn_limit}"
              upper="${wheel_turn_limit}"
              effort="0" velocity="0"/>
-      <parent link="spring2_${name}"/>
+<!--      <parent link="spring2_${name}"/>-->
+      <parent link="${base_name}"/>
       <child link="steer_${name}"/>
       <origin xyz="${xyz}" rpy="0 0 0"/>

Commit message: Fixed revolute joint

File: tigra_description/urdf/robot.urdf.xacro (robot description, xacro)
@@ -1,165 +1,111 @@
-<?xml version="1.0" ?>
+<?xml version="1.0"?>
 <robot name="tigra" xmlns:xacro="http://www.ros.org/wiki/xacro">
-<xacro:property name="length" value="1.85" />
-<xacro:property name="width" value="0.75" />
-<xacro:property name="heigth" value="0.6" />
-<xacro:property name="mass" value="420" />
-<xacro:property name="wheel_width" value="0.25" />
-<xacro:property name="wheel_radius" value="0.25" />
-<xacro:property name="wheel_mass" value="20" />
-<xacro:property name="wheel_turn_limit" value="${pi/4}"/>
-<xacro:property name="springStiffness" value="105" />
-<!-- inertia -->
-<xacro:macro name="null_inertial">
-    <inertial>
-      <mass value="0.001"/>
-      <inertia ixx="0.001" ixy="0" ixz="0"
-               iyy="0.001" iyz="0"
-               izz="0.001"/>
-    </inertial>
-</xacro:macro>
-<xacro:macro name="base_inertial"
-               params="width length height mass *origin">
-    <inertial>
-      <xacro:insert_block name="origin"/>
-      <mass value="${mass}"/>
-      <inertia ixx="${mass * (width * width + height * height) / 12}"
-               ixy="0" ixz="0"
-               iyy="${mass * (length * length + height * height) / 12}"
-               iyz="0"
-               izz="${mass * (width * width + length * length) / 12}"/>
-    </inertial>
-</xacro:macro>
-<xacro:macro name="wheel_inertial"
-               params="r h mass *origin">
-    <inertial>
-      <xacro:insert_block name="origin"/>
-      <mass value="${mass}"/>
-      <inertia ixx="${mass / 12 * (3 * r * r + h * h)}" ixy="0.0" ixz="0.0"
-               iyy="${mass / 12 * (3 * r * r + h * h)}" iyz="0.0"
-               izz="${mass / 2 * r * r}" />
-    </inertial>
-</xacro:macro>
-<!-- xacro base new -->
-<link name="base_link">
-<pose>0 0 0 0 0 0</pose>
-    <visual>
-     	<origin xyz="0 0 0" rpy="0 0 0" />
-        <geometry>
-            <box size="${length} ${width} ${heigth}"/>
-        </geometry>
-        <material name="blue"/>
-    </visual>
-    <collision name="base_collision">
-    	<origin xyz="0 0 0" rpy="0 0 0" />
-        <geometry>
-            <box size="${length} ${width} ${heigth}"/>
-        </geometry>
-    </collision>
-	<xacro:base_inertial
-    width="${width}" length="${length}"
-	height="${heigth}" mass="${mass}" >
-    <origin xyz="0 0 0" rpy="0 0 0" />
-	</xacro:base_inertial>
-</link>
-<!-- xacro wheel new -->
-<xacro:macro name="wheels" params="name">
-    <link name="${name}">
-      <visual>
-        <origin xyz="0 0 0" rpy="0 0 0" />
-        <geometry>
-          <cylinder length="${wheel_width}" radius="${wheel_radius}"/>
-        </geometry>
-      </visual>
-      <collision>
-        <origin xyz="0 0 0" rpy="0 0 0" />
-        <geometry>
-          <cylinder length="${wheel_width}" radius="${wheel_radius}"/>
-        </geometry>
-      </collision>
-      <xacro:wheel_inertial
-          r="${wheel_radius}" h="${wheel_width}"
-          mass="${wheel_mass}" >
-	  <origin xyz="0 0 0" rpy="0 0 0" />
-      </xacro:wheel_inertial>
-    </link>
-</xacro:macro>
-<!-- zawarka solution -->
-<!-- speed -->
-<xacro:macro name="speed_wheel" params="name base_name xyz ">
-    <xacro:wheels name="wheel_${name}" />
-<!--
-    <link name="spring1_${name}">
-      <xacro:null_inertial/>
-    </link>
-    <gazebo reference="${name}_spring_joint">
-    	<implicitSpringDamper>true</implicitSpringDamper>
-    	<springStiffness>${springStiffness}</springStiffness>
-    	<springReference>0</springReference>
-    </gazebo>
-    <joint name="${name}_spring_joint" type="prismatic">
-    <limit lower="-0.05" upper="0.05" effort="0" velocity="0"/>
-      <parent link="${base_name}"/>
-      <child link="spring1_${name}"/>
-	  <dynamics damping="0.0" friction="0.0"/>
-	  <axis xyz="0 0 1"/>
-    </joint>
--->
-    <joint name="${name}_speed_joint" type="continuous">
-<!--      <parent link="spring1_${name}"/> -->
-      <parent link="${base_name}"/>
-      <child link="wheel_${name}"/>
-      <origin xyz="${xyz}" rpy="${pi/2} 0 0"/>
-      <axis xyz="0 0 -1"/>
-      <limit effort="500.0" velocity="11.0" />
-    </joint>
-</xacro:macro>
-<!-- steer -->
-<xacro:macro name="steer_wheel" params="name base_name xyz">
-    <xacro:wheels name="wheel_${name}" />
-<!--
-    <link name="spring2_${name}">
-      <xacro:null_inertial/>
-    </link>
--->
-     <link name="steer_${name}">
-      <xacro:null_inertial/>
-    </link>
-<!--
-    <gazebo reference="${name}_spring_joint">
-    	<implicitSpringDamper>true</implicitSpringDamper>
-    	<springStiffness>${springStiffness}</springStiffness>
-    	<springReference>0</springReference>
-    </gazebo>
-    <joint name="${name}_spring_joint" type="prismatic">
-    <limit lower="-0.05" upper="0.05" effort="0" velocity="0"/>
-      <parent link="${base_name}"/>
-      <child link="spring2_${name}"/>
-	  <dynamics damping="0.0" friction="0.0"/>
-	  <axis xyz="0 0 1"/>
-    </joint>
--->
-    <joint name="${name}_steer_joint" type="revolute">
-      <limit lower="${-wheel_turn_limit}"
-             upper="${wheel_turn_limit}"
-             effort="0" velocity="0"/>
-<!--      <parent link="spring2_${name}"/>-->
-      <parent link="${base_name}"/>
-      <child link="steer_${name}"/>
-      <origin xyz="${xyz}" rpy="0 0 0"/>
-      <axis xyz="0 0 1"/>
-    </joint>
-    <joint name="${name}_speed_joint" type="continuous">
-      <parent link="steer_${name}"/>
-      <child link="wheel_${name}"/>
-      <origin xyz="0 0 0" rpy="${pi/2} 0 0"/>
-      <axis xyz="0 0 -1"/>
-      <limit effort="500" velocity="11.0" />
-    </joint>
-</xacro:macro>
-<!-- steer_wheel -->
+	<xacro:property name="length" value="1.85" />
+	<xacro:property name="width" value="0.75" />
+	<xacro:property name="heigth" value="0.6" />
+	<xacro:property name="mass" value="420" />
+	<xacro:property name="wheel_width" value="0.25" />
+	<xacro:property name="wheel_radius" value="0.25" />
+	<xacro:property name="wheel_mass" value="20" />
+	<xacro:property name="wheel_turn_limit" value="${pi/4}" />
+	<!-- inertia -->
+	<xacro:macro name="null_inertial">
+		<inertial>
+			<mass value="1.0" />
+			<inertia ixx="0.01" ixy="0" ixz="0" iyy="0.01" iyz="0" izz="0.01" />
+		</inertial>
+	</xacro:macro>
+	<xacro:macro name="base_inertial" params="width length height mass *origin">
+		<inertial>
+			<xacro:insert_block name="origin" />
+			<mass value="${mass}" />
+			<inertia ixx="${mass * (width * width + height * height) / 12}" ixy="0" ixz="0" iyy="${mass * (length * length + height * height) / 12}" iyz="0" izz="${mass * (width * width + length * length) / 12}" />
+		</inertial>
+	</xacro:macro>
+	<xacro:macro name="wheel_inertial" params="r h mass *origin">
+		<inertial>
+			<xacro:insert_block name="origin" />
+			<mass value="${mass}" />
+			<inertia ixx="${mass / 12 * (3 * r * r + h * h)}" ixy="0.0" ixz="0.0" iyy="${mass / 12 * (3 * r * r + h * h)}" iyz="0.0" izz="${mass / 2 * r * r}" />
+		</inertial>
+	</xacro:macro>
+	<!-- xacro base new -->
+	<link name="base_link">
+		<pose>
+			0 0 0 0 0 0
+		</pose>
+		<visual>
+			<origin xyz="0 0 0" rpy="0 0 0" />
+			<geometry>
+				<box size="${length} ${width} ${heigth}" />
+			</geometry>
+			<material name="blue" />
+		</visual>
+		<collision name="base_collision">
+			<origin xyz="0 0 0" rpy="0 0 0" />
+			<geometry>
+				<box size="${length} ${width} ${heigth}" />
+			</geometry>
+		</collision>
+		<xacro:base_inertial width="${width}" length="${length}" height="${heigth}" mass="${mass}">
+			<origin xyz="0 0 0" rpy="0 0 0" />
+		</xacro:base_inertial>
+	</link>
+	<!-- xacro wheel new -->
+	<xacro:macro name="wheels" params="name">
+		<link name="${name}">
+			<visual>
+				<origin xyz="0 0 0" rpy="${pi/2} 0 0" />
+				<geometry>
+					<cylinder length="${wheel_width}" radius="${wheel_radius}" />
+				</geometry>
+			</visual>
+			<collision>
+				<origin xyz="0 0 0" rpy="${pi/2} 0 0" />
+				<geometry>
+					<cylinder length="${wheel_width}" radius="${wheel_radius}" />
+				</geometry>
+			</collision>
+			<xacro:wheel_inertial r="${wheel_radius}" h="${wheel_width}" mass="${wheel_mass}">
+				<origin xyz="0 0 0" rpy="${pi/2} 0 0" />
+			</xacro:wheel_inertial>
+		</link>
+	</xacro:macro>
+	<!-- speed -->
+	<xacro:macro name="speed_wheel" params="name base_name xyz ">
+		<joint name="${name}_speed_joint" type="continuous">
+			<parent link="${base_name}" />
+			<child link="wheel_${name}" />
+			<origin xyz="${xyz}" rpy="0 0 0" />
+			<axis xyz="0 1 0" />
+			<limit effort="500" velocity="10" />
+		</joint>
+		<xacro:wheels name="wheel_${name}" />
+	</xacro:macro>
+  <!-- steer -->
+	<xacro:macro name="steer_wheel" params="name base_name xyz">
+		<joint name="${name}_steer_joint" type="revolute">
+			<parent link="${base_name}" />
+			<child link="steer_${name}" />
+			<origin xyz="${xyz}" rpy="0 0 0" />
+			<axis xyz="0 0 1" />
+			<limit lower="${-wheel_turn_limit}" upper="${wheel_turn_limit}" effort="0" velocity="0" />
+		</joint>
+		<link name="steer_${name}">
+			<xacro:null_inertial />
+		</link>
+		<joint name="${name}_speed_joint" type="continuous">
+			<parent link="steer_${name}" />
+			<child link="wheel_${name}" />
+			<origin xyz="0 0 0" rpy="0 0 0" />
+			<axis xyz="0 1 0" />
+			<limit effort="500" velocity="10" />
+		</joint>
+		<xacro:wheels name="wheel_${name}" />
+	</xacro:macro>
+	<!-- steer_wheel -->
 	<xacro:steer_wheel name="joint_right_wheel_1" base_name="base_link" xyz="0.5 -0.375 -0.35" />
 	<xacro:steer_wheel name="joint_left_wheel_1" base_name="base_link" xyz="0.5 0.375 -0.35" />
-<!-- speed_wheel -->
+	<!-- speed_wheel -->
 	<xacro:speed_wheel name="joint_right_wheel_2" base_name="base_link" xyz="-0.5 -0.375 -0.35" />
 	<xacro:speed_wheel name="joint_left_wheel_2" base_name="base_link" xyz="-0.5 0.375 -0.35" />
