Commit message: Update Tigra Description

File: tigra_description/urdf/robot.urdf.xacro (robot description, xacro)
@@ -32,7 +32,4 @@
 	<!-- xacro base new -->
 	<link name="base_link">
-		<pose>
-			0 0 0 0 0 0
-		</pose>
 		<visual>
 			<origin xyz="0 0 0" rpy="0 0 0" />
@@ -104,4 +101,13 @@
 		<xacro:wheels name="wheel_${name}" />
 	</xacro:macro>
+  	<gazebo>
+    		<plugin name="ModelPlugin" filename="libtigra_description.so" >
+      			<robotName>tigra</robotName>
+            <wheel_rl_joint_>joint_right_wheel_1_speed_joint</wheel_rl_joint_>
+            <wheel_rr_joint_>joint_left_wheel_1_speed_joint</wheel_rr_joint_>
+            <wheel_fl_joint_>joint_right_wheel_2_speed_joint</wheel_fl_joint_>
+            <wheel_fr_joint_>joint_left_wheel_2_speed_joint</wheel_fr_joint_>
+   		 </plugin>
+	</gazebo>
 	<!-- steer_wheel -->
 	<xacro:steer_wheel name="joint_right_wheel_1" base_name="base_link" xyz="0.5 -0.375 -0.35" />

File: tigra_description/urdf/springrobot.urdf.xacro (robot description, xacro)
@@ -4,17 +4,18 @@
 <xacro:property name="width" value="0.75" />
 <xacro:property name="heigth" value="0.6" />
-<xacro:property name="mass" value="0.42" />
+<xacro:property name="mass" value="420" />
 <xacro:property name="wheel_width" value="0.25" />
 <xacro:property name="wheel_radius" value="0.25" />
-<xacro:property name="wheel_mass" value="0.02" />
+<xacro:property name="wheel_mass" value="20" />
 <xacro:property name="wheel_turn_limit" value="${pi/4}"/>
-<xacro:property name="springStiffness" value="105" />
+<xacro:property name="springStiffness" value="125000" />
+<xacro:property name="springReference" value="0" />
 <!-- inertia -->
 <xacro:macro name="null_inertial">
     <inertial>
-      <mass value="0.001"/>
-      <inertia ixx="0.001" ixy="0" ixz="0"
-               iyy="0.001" iyz="0"
-               izz="0.001"/>
+      <mass value="1.0"/>
+      <inertia ixx="0.01" ixy="0" ixz="0"
+               iyy="0.01" iyz="0"
+               izz="0.01"/>
     </inertial>
 </xacro:macro>
@@ -43,5 +44,4 @@
 <!-- xacro base new -->
 <link name="base_link">
-<pose>0 0 0 0 0 0</pose>
     <visual>
      	<origin xyz="0 0 0" rpy="0 0 0" />
@@ -67,5 +67,5 @@
     <link name="${name}">
       <visual>
-        <origin xyz="0 0 0" rpy="0 0 0" />
+        <origin xyz="0 0 0" rpy="${pi/2} 0 0" />
         <geometry>
           <cylinder length="${wheel_width}" radius="${wheel_radius}"/>
@@ -73,5 +73,5 @@
       </visual>
       <collision>
-        <origin xyz="0 0 0" rpy="0 0 0" />
+        <origin xyz="0 0 0" rpy="${pi/2} 0 0" />
         <geometry>
           <cylinder length="${wheel_width}" radius="${wheel_radius}"/>
@@ -81,22 +81,18 @@
           r="${wheel_radius}" h="${wheel_width}"
           mass="${wheel_mass}" >
-	  <origin xyz="0 0 0" rpy="0 0 0" />
+	  <origin xyz="0 0 0" rpy="${pi/2} 0 0" />
       </xacro:wheel_inertial>
     </link>
 </xacro:macro>
-<!-- zawarka solution -->
 <!-- speed -->
 <xacro:macro name="speed_wheel" params="name base_name xyz ">
     <xacro:wheels name="wheel_${name}" />
-    <link name="spring1_${name}">
-      <xacro:null_inertial/>
-    </link>
     <gazebo reference="${name}_spring_joint">
     	<implicitSpringDamper>true</implicitSpringDamper>
     	<springStiffness>${springStiffness}</springStiffness>
-    	<springReference>0</springReference>
+    	<springReference>${springReference}</springReference>
     </gazebo>
     <joint name="${name}_spring_joint" type="prismatic">
-    <limit lower="-0.05" upper="0.05" effort="0" velocity="0"/>
+    <limit lower="-0.1" upper="0.1" effort="0" velocity="0"/>
       <parent link="${base_name}"/>
       <child link="spring1_${name}"/>
@@ -104,10 +100,13 @@
 	  <axis xyz="0 0 1"/>
     </joint>
+    <link name="spring1_${name}">
+      <xacro:null_inertial/>
+    </link>
     <joint name="${name}_speed_joint" type="continuous">
       <parent link="spring1_${name}"/>
       <child link="wheel_${name}"/>
-      <origin xyz="${xyz}" rpy="${pi/2} 0 0"/>
-      <axis xyz="0 0 -1"/>
-      <limit effort="500.0" velocity="11.0" />
+      <origin xyz="${xyz}" rpy="0 0 0"/>
+      <axis xyz="0 1 0"/>
+      <limit effort="500.0" velocity="10.0" />
     </joint>
 </xacro:macro>
@@ -115,17 +114,11 @@
 <xacro:macro name="steer_wheel" params="name base_name xyz">
     <xacro:wheels name="wheel_${name}" />
-    <link name="spring2_${name}">
-      <xacro:null_inertial/>
-    </link>
-     <link name="steer_${name}">
-      <xacro:null_inertial/>
-    </link>
     <gazebo reference="${name}_spring_joint">
     	<implicitSpringDamper>true</implicitSpringDamper>
     	<springStiffness>${springStiffness}</springStiffness>
-    	<springReference>0</springReference>
+    	<springReference>${springReference}</springReference>
     </gazebo>
     <joint name="${name}_spring_joint" type="prismatic">
-    <limit lower="-0.05" upper="0.05" effort="0" velocity="0"/>
+    <limit lower="-0.1" upper="0.1" effort="0" velocity="0"/>
       <parent link="${base_name}"/>
       <child link="spring2_${name}"/>
@@ -133,4 +126,7 @@
 	  <axis xyz="0 0 1"/>
     </joint>
+    <link name="spring2_${name}">
+      <xacro:null_inertial/>
+    </link>
     <joint name="${name}_steer_joint" type="revolute">
       <limit lower="${-wheel_turn_limit}"
@@ -142,12 +138,24 @@
       <axis xyz="0 0 1"/>
     </joint>
+     <link name="steer_${name}">
+      <xacro:null_inertial/>
+    </link>
     <joint name="${name}_speed_joint" type="continuous">
       <parent link="steer_${name}"/>
       <child link="wheel_${name}"/>
-      <origin xyz="0 0 0" rpy="${pi/2} 0 0"/>
-      <axis xyz="0 0 -1"/>
-      <limit effort="500" velocity="11.0" />
+      <origin xyz="0 0 0" rpy="0 0 0"/>
+      <axis xyz="0 1 0"/>
+      <limit effort="500" velocity="10.0" />
     </joint>
 </xacro:macro>
+  	<gazebo>
+    		<plugin name="ModelPlugin" filename="libtigra_description.so" >
+      			<robotName>tigra</robotName>
+            <wheel_rl_joint_>joint_right_wheel_1_speed_joint</wheel_rl_joint_>
+            <wheel_rr_joint_>joint_left_wheel_1_speed_joint</wheel_rr_joint_>
+            <wheel_fl_joint_>joint_right_wheel_2_speed_joint</wheel_fl_joint_>
+            <wheel_fr_joint_>joint_left_wheel_2_speed_joint</wheel_fr_joint_>
+   		 </plugin>
+	</gazebo>
 <!-- steer_wheel -->
 	<xacro:steer_wheel name="joint_right_wheel_1" base_name="base_link" xyz="0.5 -0.375 -0.35" />

Commit message: Add Labyrinth

File: tigra_description/urdf/robot.urdf.xacro (robot description, xacro)
@@ -87,5 +87,5 @@
 			<origin xyz="${xyz}" rpy="0 0 0" />
 			<axis xyz="0 0 1" />
-			<limit lower="${-wheel_turn_limit}" upper="${wheel_turn_limit}" effort="0" velocity="0" />
+			<limit lower="${-wheel_turn_limit}" upper="${wheel_turn_limit}" effort="1000" velocity="0" />
 		</joint>
 		<link name="steer_${name}">
@@ -102,10 +102,10 @@
 	</xacro:macro>
   	<gazebo>
-    		<plugin name="ModelPlugin" filename="libtigra_description.so" >
+    		<plugin name="tigra_interface_plugin" filename="libtigra_interface_plugin.so" >
       			<robotName>tigra</robotName>
-            <wheel_rl_joint_>joint_right_wheel_1_speed_joint</wheel_rl_joint_>
-            <wheel_rr_joint_>joint_left_wheel_1_speed_joint</wheel_rr_joint_>
-            <wheel_fl_joint_>joint_right_wheel_2_speed_joint</wheel_fl_joint_>
-            <wheel_fr_joint_>joint_left_wheel_2_speed_joint</wheel_fr_joint_>
+            <wheel_rl_joint_>joint_left_wheel_1_speed_joint</wheel_rl_joint_>
+            <wheel_rr_joint_>joint_right_wheel_1_speed_joint</wheel_rr_joint_>
+            <wheel_fl_joint_>joint_left_wheel_2_speed_joint</wheel_fl_joint_>
+            <wheel_fr_joint_>joint_right_wheel_2_speed_joint</wheel_fr_joint_>
    		 </plugin>
 	</gazebo>

File: tigra_description/urdf/springrobot.urdf.xacro (robot description, xacro)
@@ -132,5 +132,5 @@
       <limit lower="${-wheel_turn_limit}"
              upper="${wheel_turn_limit}"
-             effort="0" velocity="0"/>
+             effort="1000" velocity="0"/>
       <parent link="spring2_${name}"/>
       <child link="steer_${name}"/>
@@ -150,10 +150,10 @@
 </xacro:macro>
   	<gazebo>
-    		<plugin name="ModelPlugin" filename="libtigra_description.so" >
+    		<plugin name="tigra_interface_plugin" filename="libtigra_interface_plugin.so" >
       			<robotName>tigra</robotName>
-            <wheel_rl_joint_>joint_right_wheel_1_speed_joint</wheel_rl_joint_>
-            <wheel_rr_joint_>joint_left_wheel_1_speed_joint</wheel_rr_joint_>
-            <wheel_fl_joint_>joint_right_wheel_2_speed_joint</wheel_fl_joint_>
-            <wheel_fr_joint_>joint_left_wheel_2_speed_joint</wheel_fr_joint_>
+            <wheel_rl_joint_>joint_left_wheel_1_speed_joint</wheel_rl_joint_>
+            <wheel_rr_joint_>joint_right_wheel_1_speed_joint</wheel_rr_joint_>
+            <wheel_fl_joint_>joint_left_wheel_2_speed_joint</wheel_fl_joint_>
+            <wheel_fr_joint_>joint_right_wheel_2_speed_joint</wheel_fr_joint_>
    		 </plugin>
 	</gazebo>
