Commit message: Add lidar

File: tigra_description/urdf/springrobot.urdf.xacro (robot description, xacro)
@@ -8,7 +8,16 @@
 <xacro:property name="wheel_radius" value="0.25" />
 <xacro:property name="wheel_mass" value="20" />
+<xacro:property name="wheelbase" value="1.0" />
+<xacro:property name="half_wheelbase" value="${wheelbase/2}" />
+<xacro:property name="track_width" value="0.8" />
 <xacro:property name="wheel_turn_limit" value="${pi/4}"/>
+<xacro:property name="degrees_30" value="${pi/6}"/>
+<xacro:property name="mid_wheel_turn_limit" value="${degrees_30}"/>
 <xacro:property name="springStiffness" value="125000" />
 <xacro:property name="springReference" value="0" />
+<xacro:property name="lidar_mass" value="0.1" />
+<xacro:property name="lidar_height" value="0.02"/>
+<xacro:property name="lidar_radius" value="0.04"/>
+<xacro:arg name="pub_tf" default="true" />
 <!-- inertia -->
 <xacro:macro name="null_inertial">
@@ -149,13 +158,80 @@
     </joint>
 </xacro:macro>
-  	<gazebo>
-    		<plugin name="tigra_interface_plugin" filename="libtigra_interface_plugin.so" >
-      			<robotName>tigra</robotName>
-            <wheel_rl_joint_>joint_left_wheel_1_speed_joint</wheel_rl_joint_>
-            <wheel_rr_joint_>joint_right_wheel_1_speed_joint</wheel_rr_joint_>
-            <wheel_fl_joint_>joint_left_wheel_2_speed_joint</wheel_fl_joint_>
-            <wheel_fr_joint_>joint_right_wheel_2_speed_joint</wheel_fr_joint_>
-   		 </plugin>
-	</gazebo>
+<!-- lidar -->
+ <!-- Hokuyo Laser -->
+  <link name="lidar_link">
+    <xacro:wheel_inertial
+        r="${lidar_radius}" h="${lidar_height}"
+        mass="${lidar_mass}" >
+      <origin xyz="0 0 0" rpy="0 0 0" />
+    </xacro:wheel_inertial>
+    <collision>
+      <origin xyz="0 0 0" rpy="0 0 0"/>
+      <geometry>
+        <cylinder length="${lidar_height}" radius="${lidar_radius}"/>
+      </geometry>
+    </collision>
+    <visual>
+      <origin xyz="0 0 0" rpy="0 0 0"/>
+      <geometry>
+        <cylinder length="${lidar_height}" radius="${lidar_radius}"/>
+      </geometry>
+    </visual>
+  </link>
+  <gazebo reference="lidar_link">
+    <material>Gazebo/Red</material>
+    <sensor type="ray" name="head_hokuyo_sensor">
+      <pose>0 0 0 0 0 0</pose>
+      <visualize>true</visualize>
+      <update_rate>40</update_rate>
+      <ray>
+        <scan>
+          <horizontal>
+            <samples>720</samples>
+            <resolution>1</resolution>
+            <min_angle>-3.14</min_angle>
+            <max_angle>3.14</max_angle>
+          </horizontal>
+        </scan>
+        <range>
+          <min>0.10</min>
+          <max>30.0</max>
+          <resolution>0.01</resolution>
+        </range>
+        <noise>
+          <type>gaussian</type>
+          <!-- Noise parameters based on published spec for Hokuyo laser
+               achieving "+-30mm" accuracy at range < 10m.  A mean of 0.0m and
+               stddev of 0.01m will put 99.7% of samples within 0.03m of the true
+               reading. -->
+          <mean>0.0</mean>
+          <stddev>0.01</stddev>
+        </noise>
+      </ray>
+      <plugin name="gazebo_ros_head_hokuyo_controller" filename="libgazebo_ros_laser.so">
+        <topicName>/tigra_description/laser/scan</topicName>
+        <frameName>lidar_link</frameName>
+      </plugin>
+    </sensor>
+  </gazebo>
+  <joint name="lidar_joint" type="fixed">
+    <axis xyz="0 1 0" />
+    <origin xyz="0 0 0.35" rpy="0 0 0"/>
+    <parent link="base_link"/>
+    <child link="lidar_link"/>
+  </joint>
+<gazebo>
+	<plugin name="tigra_interface_plugin" filename="libtigra_interface_plugin.so" >
+		<robotName>tigra</robotName>
+		<maxSteerRad>${mid_wheel_turn_limit}</maxSteerRad>
+		<wheelbase>${wheelbase}</wheelbase>
+		<wheelRadius>${wheel_radius}</wheelRadius>
+		<trackWidth>${track_width}</trackWidth>
+		<wheel_rl_joint_>joint_left_wheel_1_speed_joint</wheel_rl_joint_>
+		<wheel_rr_joint_>joint_right_wheel_1_speed_joint</wheel_rr_joint_>
+		<wheel_fl_joint_>joint_left_wheel_2_speed_joint</wheel_fl_joint_>
+		<wheel_fr_joint_>joint_right_wheel_2_speed_joint</wheel_fr_joint_>
+	</plugin>
+</gazebo>
 <!-- steer_wheel -->
 	<xacro:steer_wheel name="joint_right_wheel_1" base_name="base_link" xyz="0.5 -0.375 -0.35" />

Commit message: Add footprint

File: tigra_description/urdf/springrobot.urdf.xacro (robot description, xacro)
@@ -19,4 +19,8 @@
 <xacro:property name="lidar_height" value="0.02"/>
 <xacro:property name="lidar_radius" value="0.04"/>
+<!-- base_footprint - base_link on floor -->
+<link name="base_footprint">
+</link>
+<gazebo reference="base_footprint"/>
 <xacro:arg name="pub_tf" default="true" />
 <!-- inertia -->
@@ -221,4 +225,10 @@
     <child link="lidar_link"/>
   </joint>
+  <joint name="base_footprint_2_link" type="fixed">
+    <parent link="base_footprint"/>
+    <child link="base_link"/>
+    <!-- base_footprint - base_link on floor -->
+    <origin xyz="0 0 ${wheel_radius}" rpy="0 0 0"/>
+  </joint>
 <gazebo>
 	<plugin name="tigra_interface_plugin" filename="libtigra_interface_plugin.so" >

Commit message: Add map

File: tigra_description/urdf/springrobot.urdf.xacro (robot description, xacro)
@@ -221,5 +221,5 @@
   <joint name="lidar_joint" type="fixed">
     <axis xyz="0 1 0" />
-    <origin xyz="0 0 0.35" rpy="0 0 0"/>
+    <origin xyz="0 0 0.55" rpy="0 0 0"/>
     <parent link="base_link"/>
     <child link="lidar_link"/>
