Commit message: #90 realsense works correctly + integrated pointcloud data into navigation

File: tigra_description/urdf/tigra_robocross21.urdf.xacro (robot description, xacro)
@@ -91,3 +91,69 @@
     </plugin>
   </gazebo>
+  <!-- Depth sensor - emulation of Intel RealSense D435 -->
+  <joint name="base_rs_camera_joint" type="fixed">
+    <parent link="base_link" />
+    <child link="rs_camera_link" />
+    <origin xyz="${body_length/2} 0 ${body_heigth/2+0.1}" rpy="0 0 0" />
+  </joint>
+  <link name="rs_camera_link">
+    <collision>
+      <origin xyz="0 0 0" rpy="0 0 0" />
+      <geometry>
+        <box size="0.02 0.2 0.02" />
+      </geometry>
+    </collision>
+    <visual>
+      <origin xyz="0 0 0" rpy="0 0 0" />
+      <geometry>
+        <box size="0.02 0.2 0.02" />
+      </geometry>
+    </visual>
+    <inertial>
+      <mass value="1e-5" />
+      <origin xyz="0 0 0" rpy="0 0 0" />
+      <inertia ixx="1e-6" ixy="0" ixz="0" iyy="1e-6" iyz="0" izz="1e-6" />
+    </inertial>
+  </link>
+  <gazebo reference="rs_camera_link">
+    <material>Gazebo/Black</material>
+    <sensor name="rs_camera_link_camera" type="depth">
+      <update_rate>20</update_rate>
+      <camera>
+        <horizontal_fov>1.3962634016</horizontal_fov>
+        <image>
+          <width>640</width>
+          <height>480</height>
+          <format>R8G8B8</format>
+        </image>
+        <clip>
+          <near>0.05</near>
+          <far>300</far>
+        </clip>
+      </camera>
+      <plugin name="camera_plugin" filename="libgazebo_ros_openni_kinect.so">
+        <baseline>0.2</baseline>
+        <alwaysOn>true</alwaysOn>
+        <updateRate>20.0</updateRate>
+        <cameraName>rs_camera</cameraName>
+        <imageTopicName>/rs_camera/color/image_raw</imageTopicName>
+        <cameraInfoTopicName>/rs_camera/color/camera_info</cameraInfoTopicName>
+        <depthImageTopicName>/rs_camera/depth/image_raw</depthImageTopicName>
+        <depthImageCameraInfoTopicName>/rs_camera/depth/camera_info</depthImageCameraInfoTopicName>
+        <pointCloudTopicName>/rs_camera/depth/color/points</pointCloudTopicName>
+        <frameName>rs_camera_optical_frame</frameName>
+        <pointCloudCutoff>0.05</pointCloudCutoff>
+        <distortionK1>0</distortionK1>
+        <distortionK2>0</distortionK2>
+        <distortionK3>0</distortionK3>
+        <distortionT1>0</distortionT1>
+        <distortionT2>0</distortionT2>
+        <CxPrime>0</CxPrime>
+        <Cx>0</Cx>
+        <Cy>0</Cy>
+        <focalLength>0</focalLength>
+        <hackBaseline>0</hackBaseline>
+      </plugin>
+    </sensor>
+  </gazebo>
 </robot>

Commit message: Local experiments (#118)
* Create Odom_intro.md

* First page Google.

* Init commit

* Update Planner_intro.md

* Update Planner_intro.md

* Update Planner_intro.md

* Delete Planner_intro.md

* Create Planner_intro.md

* Update Planner_intro.md

* Update Planner_intro.md

* Update Planner_intro.md

* Update Odom_intro.md

* Update Odom_intro.md

* Update Odom_intro.md

* README modified and fixed build script

* Removed ublox from build script

* Fixed multiple issues with sim

* Update Odom_intro.md

* rtabmap launch

* RGB-D Handheld Mapping launch. Database saved in ~/.ros/rtabmap.db.

* Update Odom_intro.md

* testing rtabmap in sim. Problems with TF.

* Create practice.md

* Files from Kuzmina T.O.

* Update practice.md

* Add files via upload

* Still problems with TF.

* Fixed TF issue

* Sim with lidar

* fixed lidar_location

* changing map launch

* tigra with lidar launch

* lidar config

* choice map or loc

* Localization error

* Reduced transform period for depth_msg conversion

* init commit

* mapping with 2d laser scan

* add transform for depth image -> laser scan

* add transform for depth image -> laser scan

* elp calibration. square 0.025

* Last fixes for repository

* charge description

* Merged develop with local_experiments

* charge description added photos

* troubles with ekf

* Updated build scripts

* added ground_truth/pose topic from gazebo

* bad imu covariance

* rtab work localization

* added ground_truth/pose topic from gazebo

* rtabmap on CPU?

* Update full_start_joy_mapping.launch

* added xiaomi head calib

* small refactor

* multiply rs_cameras rtabmap

* Delete download_docs.sh

* Updated model, deprecated some files

* Small readme update

* added asphalt model

* sim works

* deleted old calib

* added sim_rtabmap

* rename rs to left&right

* added start_rtabmap_multi

* rtab arguments for multicam

* rtabmap gen_scan mode only

* added moving_base cfgs gps

* pepelac experiments

* added ekf global

* Updated scripts

* rtab work with gps

* Updated tigra model

Co-authored-by: ashenone23 <91793116+ashenone23@users.noreply.github.com>
Co-authored-by: DepartmentNotebookUser <dep-nb-user@mail.ru>
Co-authored-by: KaiL4eK <darklexi494@gmail.com>
Co-authored-by: KaiL4eK <alexey4dev@gmail.com>
Co-authored-by: tigra <tigra@etu.ru>
Co-authored-by: Alex Home WSL <alex_home_wsl@example.com>
Co-authored-by: aligtr <aligtr@bk.ru>
Co-authored-by: Alexey Devyatkin <nine-4lex@mail.ru>
Co-authored-by: ashenone23 <devil2309@yandex.ru>

File: tigra_description/urdf/tigra_robocross21.urdf.xacro (robot description, xacro)
@@ -1,53 +1,12 @@
 <?xml version="1.0"?>
 <robot name="tigra" xmlns:xacro="http://www.ros.org/wiki/xacro">
-  <xacro:include filename="$(find tigra_description)/urdf/tigra.urdf.xacro" />
-  <!-- IMU -->
-  <link name="imu_link">
-    <visual>
-      <geometry>
-        <box size="${imu_length} 0.2 ${imu_height}" />
-      </geometry>
-    </visual>
-    <collision>
-      <geometry>
-        <box size="${imu_length} 0.2 ${imu_height}" />
-      </geometry>
-    </collision>
-    <inertial>
-      <mass value="1e-5" />
-      <origin xyz="0 0 0" rpy="0 0 0" />
-      <inertia ixx="1e-6" ixy="0" ixz="0" iyy="1e-6" iyz="0" izz="1e-6" />
-    </inertial>
-  </link>
-  <joint name="base_imu_joint" type="fixed">
-    <parent link="base_link" />
-    <child link="imu_link" />
-    <origin xyz="${body_length/2-imu_length/2} 0 ${body_heigth/2+imu_height/2}" rpy="0 0 0" />
-  </joint>
-  <gazebo reference="imu_link">
-    <material>Gazebo/Red</material>
-    <gravity>true</gravity>
-    <sensor name="imu_sensor" type="imu">
-      <always_on>true</always_on>
-      <update_rate>100</update_rate>
-      <visualize>true</visualize>
-      <topic>__default_topic__</topic>
-      <plugin filename="libgazebo_ros_imu_sensor.so" name="imu_plugin">
-        <topicName>$(arg robot_name)/imu</topicName>
-        <bodyName>imu_link</bodyName>
-        <updateRateHZ>20.0</updateRateHZ>
-        <gaussianNoise>0.0</gaussianNoise>
-        <xyzOffset>0 0 0</xyzOffset>
-        <rpyOffset>0 0 0</rpyOffset>
-        <frameName>imu_link</frameName>
-      </plugin>
-      <pose>0 0 0 0 0 0</pose>
-    </sensor>
-  </gazebo>
+  <xacro:include filename="$(find tigra_description)/urdf/base.urdf.xacro" />
+	<xacro:include filename="$(find maddrive_urdf_tools)/urdf/macros/realsense.urdf.xacro" />
+	<xacro:include filename="$(find maddrive_urdf_tools)/urdf/macros/elp_stereo.urdf.xacro" />
   <!-- GPS -->
   <joint name="base_gps_joint" type="fixed">
     <parent link="base_link" />
     <child link="gps_link" />
-    <origin xyz="0 0 ${body_heigth/2+imu_height/2}" rpy="0 0 0" />
+    <origin xyz="0 0 ${body_heigth/2+0.1}" rpy="0 0 0" />
   </joint>
   <link name="gps_link">
@@ -90,71 +49,24 @@
       <velocityGaussianNoise>0.5 0.5 0.5</velocityGaussianNoise>
     </plugin>
+    <plugin name="p3d_base_controller" filename="libgazebo_ros_p3d.so">
+      <alwaysOn>true</alwaysOn>
+      <updateRate>50.0</updateRate>
+      <bodyName>base_link</bodyName>
+      <topicName>ground_truth/state</topicName>
+      <gaussianNoise>0.01</gaussianNoise>
+      <frameName>world</frameName>
+      <xyzOffsets>0 0 0</xyzOffsets>
+      <rpyOffsets>0 0 0</rpyOffsets>
+    </plugin>
   </gazebo>
-  <!-- Depth sensor - emulation of Intel RealSense D435 -->
-  <joint name="base_rs_camera_joint" type="fixed">
-    <parent link="base_link" />
-    <child link="rs_camera_link" />
-    <origin xyz="${body_length/2} 0 ${body_heigth/2+0.1}" rpy="0 0 0" />
-  </joint>
-  <link name="rs_camera_link">
-    <collision>
-      <origin xyz="0 0 0" rpy="0 0 0" />
-      <geometry>
-        <box size="0.02 0.2 0.02" />
-      </geometry>
-    </collision>
-    <visual>
-      <origin xyz="0 0 0" rpy="0 0 0" />
-      <geometry>
-        <box size="0.02 0.2 0.02" />
-      </geometry>
-    </visual>
-    <inertial>
-      <mass value="1e-5" />
-      <origin xyz="0 0 0" rpy="0 0 0" />
-      <inertia ixx="1e-6" ixy="0" ixz="0" iyy="1e-6" iyz="0" izz="1e-6" />
-    </inertial>
-  </link>
-  <gazebo reference="rs_camera_link">
-    <material>Gazebo/Black</material>
-    <sensor name="rs_camera_link_camera" type="depth">
-      <update_rate>20</update_rate>
-      <camera>
-        <horizontal_fov>1.3962634016</horizontal_fov>
-        <image>
-          <width>640</width>
-          <height>480</height>
-          <format>R8G8B8</format>
-        </image>
-        <clip>
-          <near>0.05</near>
-          <far>300</far>
-        </clip>
-      </camera>
-      <plugin name="camera_plugin" filename="libgazebo_ros_openni_kinect.so">
-        <baseline>0.2</baseline>
-        <alwaysOn>true</alwaysOn>
-        <updateRate>20.0</updateRate>
-        <cameraName>rs_camera</cameraName>
-        <imageTopicName>/rs_camera/color/image_raw</imageTopicName>
-        <cameraInfoTopicName>/rs_camera/color/camera_info</cameraInfoTopicName>
-        <depthImageTopicName>/rs_camera/depth/image_raw</depthImageTopicName>
-        <depthImageCameraInfoTopicName>/rs_camera/depth/camera_info</depthImageCameraInfoTopicName>
-        <pointCloudTopicName>/rs_camera/depth/color/points</pointCloudTopicName>
-        <frameName>rs_camera_optical_frame</frameName>
-        <pointCloudCutoff>0.05</pointCloudCutoff>
-        <pointCloudCutoffMax>10</pointCloudCutoffMax>
-        <distortionK1>0</distortionK1>
-        <distortionK2>0</distortionK2>
-        <distortionK3>0</distortionK3>
-        <distortionT1>0</distortionT1>
-        <distortionT2>0</distortionT2>
-        <CxPrime>0</CxPrime>
-        <Cx>0</Cx>
-        <Cy>0</Cy>
-        <focalLength>0</focalLength>
-        <hackBaseline>0</hackBaseline>
-      </plugin>
-    </sensor>
-  </gazebo>
+	<xacro:realsense_435
+			name="rs_camera"
+			base_link_name="base_link"
+			xyz="${body_length/2} 0 ${body_heigth/2+0.1}"
+			rpy="0 0 0" />
+  <xacro:elp_stereo
+			name="elp_stereo"
+			base_link_name="base_link"
+			xyz="-${body_length/2-wheelbase/2+0.05} 0 0"
+			rpy="0 0 ${pi}" />
 </robot>
