Commit message: Updated tigra model

File: tigra_description/urdf/params.urdf.xacro (robot description, xacro)
@@ -17,6 +17,4 @@
     <xacro:property name="lidar_location" value="${body_heigth/2+0.01}" />
     <xacro:property name="gps_height" value="0.05" />
-    <xacro:property name="imu_height" value="0.05" />
-    <xacro:property name="imu_length" value="0.2" />
     <xacro:property name="odom_frame" value="odom_wheel" />
     <xacro:arg name="pub_tf" default="true" />

File: tigra_description/urdf/tigra_robocross21.urdf.xacro (robot description, xacro)
@@ -3,52 +3,10 @@
   <xacro:include filename="$(find tigra_description)/urdf/base.urdf.xacro" />
 	<xacro:include filename="$(find maddrive_urdf_tools)/urdf/macros/realsense.urdf.xacro" />
-  <!-- IMU -->
-  <link name="imu_link">
-    <visual>
-      <geometry>
-        <box size="${imu_length} 0.2 ${imu_height}" />
-      </geometry>
-    </visual>
-    <collision>
-      <geometry>
-        <box size="${imu_length} 0.2 ${imu_height}" />
-      </geometry>
-    </collision>
-    <inertial>
-      <mass value="1e-5" />
-      <origin xyz="0 0 0" rpy="0 0 0" />
-      <inertia ixx="1e-6" ixy="0" ixz="0" iyy="1e-6" iyz="0" izz="1e-6" />
-    </inertial>
-  </link>
-  <joint name="base_imu_joint" type="fixed">
-    <parent link="base_link" />
-    <child link="imu_link" />
-    <origin xyz="${body_length/2-imu_length/2} 0 ${body_heigth/2+imu_height/2}" rpy="0 0 0" />
-  </joint>
-  <gazebo reference="imu_link">
-    <material>Gazebo/Red</material>
-    <gravity>true</gravity>
-    <sensor name="imu_sensor" type="imu">
-      <always_on>true</always_on>
-      <update_rate>100</update_rate>
-      <visualize>true</visualize>
-      <topic>__default_topic__</topic>
-      <plugin filename="libgazebo_ros_imu_sensor.so" name="imu_plugin">
-        <topicName>$(arg robot_name)/imu</topicName>
-        <bodyName>imu_link</bodyName>
-        <updateRateHZ>20.0</updateRateHZ>
-        <gaussianNoise>0.0</gaussianNoise>
-        <xyzOffset>0 0 0</xyzOffset>
-        <rpyOffset>0 0 0</rpyOffset>
-        <frameName>imu_link</frameName>
-      </plugin>
-      <pose>0 0 0 0 0 0</pose>
-    </sensor>
-  </gazebo>
+	<xacro:include filename="$(find maddrive_urdf_tools)/urdf/macros/elp_stereo.urdf.xacro" />
   <!-- GPS -->
   <joint name="base_gps_joint" type="fixed">
     <parent link="base_link" />
     <child link="gps_link" />
-    <origin xyz="0 0 ${body_heigth/2+imu_height/2}" rpy="0 0 0" />
+    <origin xyz="0 0 ${body_heigth/2+0.1}" rpy="0 0 0" />
   </joint>
   <link name="gps_link">
@@ -107,3 +65,8 @@
 			xyz="${body_length/2} 0 ${body_heigth/2+0.1}"
 			rpy="0 0 0" />
+  <xacro:elp_stereo
+			name="elp_stereo"
+			base_link_name="base_link"
+			xyz="-${body_length/2-wheelbase/2+0.05} 0 0"
+			rpy="0 0 ${pi}" />
 </robot>

Commit message: вытащил описание gps в ros_shared + под обновленные макросы камер подстроил парметры

File: tigra_description/urdf/params.urdf.xacro (robot description, xacro)
@@ -16,5 +16,4 @@
     <xacro:property name="track_width" value="${props['track_width']}" />
     <xacro:property name="lidar_location" value="${body_heigth/2+0.01}" />
-    <xacro:property name="gps_height" value="0.05" />
     <xacro:property name="odom_frame" value="odom_wheel" />
     <xacro:arg name="pub_tf" default="true" />

File: tigra_description/urdf/tigra_robocross21.urdf.xacro (robot description, xacro)
@@ -4,68 +4,17 @@
 	<xacro:include filename="$(find maddrive_urdf_tools)/urdf/macros/realsense.urdf.xacro" />
 	<xacro:include filename="$(find maddrive_urdf_tools)/urdf/macros/elp_stereo.urdf.xacro" />
-  <!-- GPS -->
-  <joint name="base_gps_joint" type="fixed">
-    <parent link="base_link" />
-    <child link="gps_link" />
-    <origin xyz="0 0 ${body_heigth/2+0.1}" rpy="0 0 0" />
-  </joint>
-  <link name="gps_link">
-    <collision>
-      <origin xyz="0 0 0" rpy="0 0 0" />
-      <geometry>
-        <box size="0.2 0.2 ${gps_height}" />
-      </geometry>
-    </collision>
-    <visual>
-      <origin xyz="0 0 0" rpy="0 0 0" />
-      <geometry>
-        <box size="0.2 0.2 ${gps_height}" />
-      </geometry>
-    </visual>
-    <inertial>
-      <mass value="1e-5" />
-      <origin xyz="0 0 0" rpy="0 0 0" />
-      <inertia ixx="1e-6" ixy="0" ixz="0" iyy="1e-6" iyz="0" izz="1e-6" />
-    </inertial>
-  </link>
-  <gazebo reference="gps_link">
-    <material>Gazebo/Orange</material>
-  </gazebo>
-  <gazebo>
-    <plugin name="gazebo_ros_gps" filename="libhector_gazebo_ros_gps.so">
-      <updateRate>4.0</updateRate>
-      <bodyName>gps_link</bodyName>
-      <frameId>gps_link</frameId>
-      <topicName>/gps/fix</topicName>
-      <velocityTopicName>/gps/fix_velocity</velocityTopicName>
-      <referenceLatitude>-30.06022459407145675</referenceLatitude>
-      <referenceLongitude>-51.173913575780311191</referenceLongitude>
-      <referenceHeading>90</referenceHeading>
-      <referenceAltitude>10</referenceAltitude>
-      <offset>0 0 0</offset>
-      <drift>0.001 0.001 0.001</drift>
-      <gaussianNoise>0.05 0.05 0.05</gaussianNoise>
-      <velocityDrift>0.001 0.001 0.001</velocityDrift>
-      <velocityGaussianNoise>0.5 0.5 0.5</velocityGaussianNoise>
-    </plugin>
-    <plugin name="p3d_base_controller" filename="libgazebo_ros_p3d.so">
-      <alwaysOn>true</alwaysOn>
-      <updateRate>50.0</updateRate>
-      <bodyName>base_link</bodyName>
-      <topicName>ground_truth/state</topicName>
-      <gaussianNoise>0.01</gaussianNoise>
-      <frameName>world</frameName>
-      <xyzOffsets>0 0 0</xyzOffsets>
-      <rpyOffsets>0 0 0</rpyOffsets>
-    </plugin>
-  </gazebo>
+  <xacro:include filename="$(find maddrive_urdf_tools)/urdf/macros/gps.urdf.xacro" />
+  <xacro:gps
+			parent="base_link"
+			origin_xyz="0 0 ${body_heigth/2+0.1}"
+			origin_rpy="0 0 0" />
 	<xacro:realsense_435
 			name="rs_camera"
-			base_link_name="base_link"
+			parent="base_link"
 			xyz="${body_length/2} 0 ${body_heigth/2+0.1}"
 			rpy="0 0 0" />
   <xacro:elp_stereo
 			name="elp_stereo"
-			base_link_name="base_link"
+			parent="base_link"
 			xyz="-${body_length/2-wheelbase/2+0.05} 0 0"
 			rpy="0 0 ${pi}" />
