Commit message: Updated model, deprecated some files

File: tigra_description/urdf/base.urdf.xacro (robot description, xacro)
@@ -1,7 +1,7 @@
 <?xml version="1.0"?>
 <robot name="tigra" xmlns:xacro="http://www.ros.org/wiki/xacro">
-	<xacro:include filename="$(find tigra_description)/urdf/macros/tigra_params.urdf.xacro" />
-	<xacro:include filename="$(find tigra_description)/urdf/macros/wheels.urdf.xacro" />
-	<xacro:include filename="$(find tigra_description)/urdf/macros/inertia.urdf.xacro" />
+	<xacro:include filename="$(find tigra_description)/urdf/params.urdf.xacro" />
+	<xacro:include filename="$(find maddrive_urdf_tools)/urdf/macros/wheels.urdf.xacro" />
+	<xacro:include filename="$(find maddrive_urdf_tools)/urdf/macros/inertia.urdf.xacro" />
 	<link name="base_link">
 		<visual>
@@ -29,4 +29,8 @@
 		<origin xyz="0 0 ${wheel_radius+wheel_shift_z}" rpy="0 0 0" />
 	</joint>
+	<xacro:steer_wheel name="front_right_wheel" base_name="base_link" xyz="${wheelbase/2} -${track_width/2} -${wheel_shift_z}" steer_limit="${wheel_turn_limit}" />
+	<xacro:steer_wheel name="front_left_wheel" base_name="base_link" xyz="${wheelbase/2} ${track_width/2} -${wheel_shift_z}" steer_limit="${wheel_turn_limit}" />
+	<xacro:speed_wheel name="rear_right_wheel" base_name="base_link" xyz="-${wheelbase/2} -${track_width/2} -${wheel_shift_z}" />
+	<xacro:speed_wheel name="rear_left_wheel" base_name="base_link" xyz="-${wheelbase/2} ${track_width/2} -${wheel_shift_z}" />
     <gazebo>
         <plugin name="tigra_interface_plugin" filename="libackermann_raw_controller_plugin.so">
@@ -40,7 +44,3 @@
         </plugin>
     </gazebo>
-	<xacro:steer_wheel name="front_right_wheel" base_name="base_link" xyz="${wheelbase/2} -${track_width/2} -${wheel_shift_z}" />
-	<xacro:steer_wheel name="front_left_wheel" base_name="base_link" xyz="${wheelbase/2} ${track_width/2} -${wheel_shift_z}" />
-	<xacro:speed_wheel name="rear_right_wheel" base_name="base_link" xyz="-${wheelbase/2} -${track_width/2} -${wheel_shift_z}" />
-	<xacro:speed_wheel name="rear_left_wheel" base_name="base_link" xyz="-${wheelbase/2} ${track_width/2} -${wheel_shift_z}" />
 </robot>

File: tigra_description/urdf/params.urdf.xacro (robot description, xacro)
@@ -2,5 +2,5 @@
 <robot xmlns:xacro="http://www.ros.org/wiki/xacro">
     <xacro:property name="yaml_file" value="$(find tigra_description)/config/props.yaml" />
-    <xacro:property name="props" value="${load_yaml(yaml_file)}" />
+    <xacro:property name="props" value="${xacro.load_yaml(yaml_file)}" />
     <xacro:property name="body_length" value="1.85" />
     <xacro:property name="body_width" value="0.75" />

File: tigra_description/urdf/tigra_robocross21.urdf.xacro (robot description, xacro)
@@ -1,5 +1,6 @@
 <?xml version="1.0"?>
 <robot name="tigra" xmlns:xacro="http://www.ros.org/wiki/xacro">
-  <xacro:include filename="$(find tigra_description)/urdf/tigra.urdf.xacro" />
+  <xacro:include filename="$(find tigra_description)/urdf/base.urdf.xacro" />
+	<xacro:include filename="$(find maddrive_urdf_tools)/urdf/macros/realsense.urdf.xacro" />
   <!-- IMU -->
   <link name="imu_link">
@@ -101,70 +102,8 @@
     </plugin>
   </gazebo>
-  <!-- Depth sensor - emulation of Intel RealSense D435 -->
-  <joint name="base_rs_camera_joint" type="fixed">
-    <parent link="base_link" />
-    <child link="rs_camera_link" />
-    <origin xyz="${body_length/2} 0 ${body_heigth/2+0.1}" rpy="0 0 0" />
-  </joint>
-  <link name="rs_camera_link">
-    <collision>
-      <origin xyz="0 0 0" rpy="0 0 0" />
-      <geometry>
-        <box size="0.02 0.2 0.02" />
-      </geometry>
-    </collision>
-    <visual>
-      <origin xyz="0 0 0" rpy="0 0 0" />
-      <geometry>
-        <box size="0.02 0.2 0.02" />
-      </geometry>
-    </visual>
-    <inertial>
-      <mass value="1e-5" />
-      <origin xyz="0 0 0" rpy="0 0 0" />
-      <inertia ixx="1e-6" ixy="0" ixz="0" iyy="1e-6" iyz="0" izz="1e-6" />
-    </inertial>
-  </link>
-  <gazebo reference="rs_camera_link">
-    <material>Gazebo/Black</material>
-    <sensor name="rs_camera_link_camera" type="depth">
-      <update_rate>20</update_rate>
-      <camera>
-        <horizontal_fov>1.3962634016</horizontal_fov>
-        <image>
-          <width>640</width>
-          <height>480</height>
-          <format>R8G8B8</format>
-        </image>
-        <clip>
-          <near>0.05</near>
-          <far>300</far>
-        </clip>
-      </camera>
-      <plugin name="camera_plugin" filename="libgazebo_ros_openni_kinect.so">
-        <baseline>0.2</baseline>
-        <alwaysOn>true</alwaysOn>
-        <updateRate>20.0</updateRate>
-        <cameraName>rs_camera</cameraName>
-        <imageTopicName>/rs_camera/color/image_raw</imageTopicName>
-        <cameraInfoTopicName>/rs_camera/color/camera_info</cameraInfoTopicName>
-        <depthImageTopicName>/rs_camera/depth/image_raw</depthImageTopicName>
-        <depthImageCameraInfoTopicName>/rs_camera/depth/camera_info</depthImageCameraInfoTopicName>
-        <pointCloudTopicName>/rs_camera/depth/color/points</pointCloudTopicName>
-        <frameName>rs_camera_optical_frame</frameName>
-        <pointCloudCutoff>0.05</pointCloudCutoff>
-        <pointCloudCutoffMax>10</pointCloudCutoffMax>
-        <distortionK1>0</distortionK1>
-        <distortionK2>0</distortionK2>
-        <distortionK3>0</distortionK3>
-        <distortionT1>0</distortionT1>
-        <distortionT2>0</distortionT2>
-        <CxPrime>0</CxPrime>
-        <Cx>0</Cx>
-        <Cy>0</Cy>
-        <focalLength>0</focalLength>
-        <hackBaseline>0</hackBaseline>
-      </plugin>
-    </sensor>
-  </gazebo>
+	<xacro:realsense_435
+			name="rs_camera"
+			base_link_name="base_link"
+			xyz="${body_length/2} 0 ${body_heigth/2+0.1}"
+			rpy="0 0 0" />
 </robot>

File: tigra_description/urdf/tigra_w_lidar.urdf.xacro (robot description, xacro)
@@ -2,5 +2,5 @@
 <robot name="tigra" xmlns:xacro="http://www.ros.org/wiki/xacro">
 	<xacro:include filename="$(find tigra_description)/urdf/tigra.urdf.xacro" />
-	<xacro:include filename="$(find tigra_description)/urdf/macros/lidar.urdf.xacro" />
+	<xacro:include filename="$(find maddrive_urdf_tools)/urdf/macros/lidar.urdf.xacro" />
 	<xacro:simple_lidar name="lidar_link" base_name="base_link" place_height="${lidar_location}" />
 </robot>

Commit message: переделал описание под шаблон "сочленение - деталь"

File: tigra_description/urdf/base.urdf.xacro (robot description, xacro)
@@ -4,4 +4,18 @@
 	<xacro:include filename="$(find maddrive_urdf_tools)/urdf/macros/wheels.urdf.xacro" />
 	<xacro:include filename="$(find maddrive_urdf_tools)/urdf/macros/inertia.urdf.xacro" />
+	<xacro:include filename="$(find maddrive_urdf_tools)/urdf/macros/common.urdf.xacro" />
+	<!-- BASE FOOTPRINT-->
+	<link name="base_footprint">
+		<xacro:null_visual/>
+		<xacro:null_collision/>
+		<xacro:null_inertia/>
+	</link>
+	<gazebo reference="base_footprint" />
+	<!-- BASE LINK-->
+	<joint name="base_footprint_2_base_link" type="fixed">
+		<parent link="base_footprint" />
+		<child link="base_link" />
+		<origin xyz="0 0 ${wheel_radius+wheel_shift_z}" rpy="0 0 0" />
+	</joint>
 	<link name="base_link">
 		<visual>
@@ -21,12 +35,5 @@
 		</xacro:box_inertia>
 	</link>
-	<!-- BASE FOOTPRINT-->
-	<link name="base_footprint" />
-	<gazebo reference="base_footprint" />
-	<joint name="base_footprint_2_link" type="fixed">
-		<parent link="base_footprint" />
-		<child link="base_link" />
-		<origin xyz="0 0 ${wheel_radius+wheel_shift_z}" rpy="0 0 0" />
-	</joint>
+	<!-- WHEELS-->
 	<xacro:steer_wheel
 		prefix="front_right"

Commit message: добавил модельку тигры

File: tigra_description/urdf/base.urdf.xacro (robot description, xacro)
@@ -22,5 +22,5 @@
 			<origin xyz="0 0 0" rpy="0 0 0" />
 			<geometry>
-				<box size="${body_length} ${body_width} ${body_heigth}" />
+				<mesh filename="package://tigra_description/meshes/quadro.dae" />
 			</geometry>
 		</visual>

Commit message: made the description of the coordinate systems of the real and simulator robot closer

File: tigra_description/urdf/base.urdf.xacro (robot description, xacro)
@@ -12,9 +12,9 @@
 	</link>
 	<gazebo reference="base_footprint" />
-	<!-- BASE LINK-->
+	<!-- BASE LINK -->
 	<joint name="base_footprint_2_base_link" type="fixed">
 		<parent link="base_footprint" />
 		<child link="base_link" />
-		<origin xyz="0 0 ${wheel_radius+wheel_shift_z}" rpy="0 0 0" />
+		<origin xyz="0 0 ${wheel_radius}" rpy="0 0 0" />
 	</joint>
 	<link name="base_link">
@@ -26,32 +26,58 @@
 		</visual>
 		<collision name="base_collision">
-			<origin xyz="0 0 0" rpy="0 0 0" />
+			<origin xyz="${body_length/2-rear_wheel_2_rear_bumper} 0 ${body_heigth/2}" rpy="0 0 0" />
 			<geometry>
 				<box size="${body_length} ${body_width} ${body_heigth}" />
 			</geometry>
 		</collision>
-		<xacro:box_inertia width="${body_width}" length="${body_length}" height="${body_heigth}" mass="${body_mass}">
-			<origin xyz="0 0 0" rpy="0 0 0" />
+		<xacro:box_inertia
+			width="${body_width}"
+			length="${body_length}"
+			height="${body_heigth}"
+			mass="${body_mass}">
+			<origin xyz="${body_length/2-rear_wheel_2_rear_bumper} 0 ${body_heigth/2}" rpy="0 0 0" />
 		</xacro:box_inertia>
 	</link>
-	<!-- WHEELS-->
+	<!-- REAR AXIS LINK -->
+	<joint name="base_footprint_2_rear_axis_link" type="fixed">
+		<parent link="base_link" />
+		<child link="rear_axis_link" />
+		<origin xyz="0 0 0" rpy="0 0 0" />
+	</joint>
+	<link name="rear_axis_link">
+		<xacro:null_visual/>
+		<xacro:null_collision/>
+		<xacro:null_inertia/>
+	</link>
+	<!-- FRONT AXIS LINK -->
+	<joint name="rear_axis_link_2_front_axis_link" type="fixed">
+		<parent link="rear_axis_link" />
+		<child link="front_axis_link" />
+		<origin xyz="${wheelbase} 0 0" rpy="0 0 0" />
+	</joint>
+	<link name="front_axis_link">
+		<xacro:null_visual/>
+		<xacro:null_collision/>
+		<xacro:null_inertia/>
+	</link>
+	<!-- WHEELS -->
 	<xacro:steer_wheel
 		prefix="front_right"
-		parent="base_link"
-		steer_origin_xyz="${wheelbase/2} -${track_width/2} -${wheel_shift_z}"
+		parent="front_axis_link"
+		steer_origin_xyz="0 -${track_width/2} 0"
 		steer_limit="${wheel_turn_limit}" />
 	<xacro:steer_wheel
 		prefix="front_left"
-		parent="base_link"
-		steer_origin_xyz="${wheelbase/2} ${track_width/2} -${wheel_shift_z}"
+		parent="front_axis_link"
+		steer_origin_xyz="0 ${track_width/2} 0"
 		steer_limit="${wheel_turn_limit}" />
 	<xacro:speed_wheel
 		prefix="rear_right"
-		parent="base_link"
-		origin_xyz="-${wheelbase/2} -${track_width/2} -${wheel_shift_z}" />
+		parent="rear_axis_link"
+		origin_xyz="0 -${track_width/2} 0" />
 	<xacro:speed_wheel
 		prefix="rear_left"
-		parent="base_link"
-		origin_xyz="-${wheelbase/2} ${track_width/2} -${wheel_shift_z}" />
+		parent="rear_axis_link"
+		origin_xyz="0 ${track_width/2} 0" />
     <gazebo>
         <plugin name="tigra_interface_plugin" filename="libackermann_raw_controller_plugin.so">

File: tigra_description/urdf/params.urdf.xacro (robot description, xacro)
@@ -1,21 +1,21 @@
 <?xml version="1.0"?>
 <robot xmlns:xacro="http://www.ros.org/wiki/xacro">
+    <xacro:arg name="robot_name" default="tigra" />
     <xacro:property name="yaml_file" value="$(find tigra_description)/config/props.yaml" />
     <xacro:property name="props" value="${xacro.load_yaml(yaml_file)}" />
-    <xacro:property name="body_length" value="1.85" />
+    <xacro:property name="front_wheel_2_front_bumper" value="0.3" />
+    <xacro:property name="rear_wheel_2_rear_bumper" value="0.3" />
+    <xacro:property name="wheelbase" value="${props['wheelbase']}" />
+    <xacro:property name="track_width" value="${props['track_width']}" />
+    <!-- основные габариты -->
+    <xacro:property name="body_length" value="${front_wheel_2_front_bumper+wheelbase+rear_wheel_2_rear_bumper}" />
     <xacro:property name="body_width" value="0.75" />
     <xacro:property name="body_heigth" value="0.6" />
     <xacro:property name="body_mass" value="340" />
+    <!-- габариты колес -->
     <xacro:property name="wheel_width" value="0.25" />
     <xacro:property name="wheel_radius" value="${props['wheel_radius']}" />
     <xacro:property name="wheel_mass" value="20" />
     <xacro:property name="wheel_turn_limit" value="${pi/4}" />
-    <xacro:property name="wheel_shift_z" value="0.35" />
-    <xacro:property name="wheelbase" value="${props['wheelbase']}" />
-    <xacro:property name="half_wheelbase" value="${wheelbase/2}" />
-    <xacro:property name="track_width" value="${props['track_width']}" />
-    <xacro:property name="lidar_location" value="${body_heigth/2+0.01}" />
-    <xacro:property name="odom_frame" value="odom_wheel" />
-    <xacro:arg name="pub_tf" default="true" />
-    <xacro:arg name="robot_name" default="tigra" />
+    <xacro:property name="wheel_shift_z" value="0.35" /> <!-- расстояние по оси Z между передней осью и осью вращения колеса -->
 </robot>

File: tigra_description/urdf/tigra_robocross21.urdf.xacro (robot description, xacro)
@@ -3,19 +3,33 @@
 	<xacro:include filename="$(find tigra_description)/urdf/base.urdf.xacro" />
 	<xacro:include filename="$(find maddrive_urdf_tools)/urdf/macros/realsense.urdf.xacro" />
-	<xacro:include filename="$(find maddrive_urdf_tools)/urdf/macros/elp_stereo.urdf.xacro" />
-	<xacro:include filename="$(find maddrive_urdf_tools)/urdf/macros/gps.urdf.xacro" />
-	<xacro:gps
+	<xacro:include filename="$(find maddrive_urdf_tools)/urdf/macros/sector_lidar.urdf.xacro" />
+	<!-- <xacro:include filename="$(find maddrive_urdf_tools)/urdf/macros/elp_stereo.urdf.xacro" /> -->
+	<!-- <xacro:include filename="$(find maddrive_urdf_tools)/urdf/macros/gps.urdf.xacro" /> -->
+	<!-- <xacro:gps
 		parent="base_link"
 		origin_xyz="0 0 ${body_heigth/2+0.1}"
-		origin_rpy="0 0 0" />
-	<xacro:realsense_435
-		name="rs_camera"
-		parent="base_link"
-		xyz="${body_length/2} 0 ${body_heigth/2+0.1}"
-		rpy="0 0 0" />
-	<xacro:elp_stereo
+		origin_rpy="0 0 0" /> -->
+	<xacro:rs_camera
+		prefix="front"
+		model="rs455"
+		parent="front_axis_link"
+		origin_xyz="-0.19 0.0 1.35"
+		origin_rpy="0.0 0.15 -0.02" />
+	<xacro:rs_camera
+		prefix="rear"
+		model="rs435"
+		parent="rear_axis_link"
+		origin_xyz="-0.19 0.0 0.61"
+		origin_rpy="3.1415 -0.01 3.1415" />
+	<!-- <xacro:sector_lidar
+		prefix="front"
+		model="c16"
+		parent="front_axis_link"
+		origin_xyz="0.07 0.0 0.715"
+		origin_rpy="1.530796327 0.0 0.04" /> -->
+	<!-- <xacro:elp_stereo
 		name="elp_stereo"
 		parent="base_link"
 		xyz="-${body_length/2-wheelbase/2+0.05} 0 0"
-		rpy="0 0 ${pi}" />
+		rpy="0 0 ${pi}" /> -->
 </robot>

Commit message: fixed an error in the joint name + removed an unused model parameter

File: tigra_description/urdf/base.urdf.xacro (robot description, xacro)
@@ -40,5 +40,5 @@
 	</link>
 	<!-- REAR AXIS LINK -->
-	<joint name="base_footprint_2_rear_axis_link" type="fixed">
+	<joint name="base_link_2_rear_axis_link" type="fixed">
 		<parent link="base_link" />
 		<child link="rear_axis_link" />

File: tigra_description/urdf/params.urdf.xacro (robot description, xacro)
@@ -18,4 +18,3 @@
     <xacro:property name="wheel_mass" value="20" />
     <xacro:property name="wheel_turn_limit" value="${pi/4}" />
-    <xacro:property name="wheel_shift_z" value="0.35" /> <!-- расстояние по оси Z между передней осью и осью вращения колеса -->
 </robot>

Commit message: little fixes in robot description and launch structure

File: tigra_description/urdf/base.urdf.xacro (robot description, xacro)
@@ -65,19 +65,23 @@
 		prefix="front_right"
 		parent="front_axis_link"
-		steer_origin_xyz="0 -${track_width/2} 0"
-		steer_limit="${wheel_turn_limit}" />
+		suspension_origin_xyz="0 -${track_width/2} 0"
+		suspension_height="${suspension_height}"
+		steer_limit="${steer_limit}" />
 	<xacro:steer_wheel
 		prefix="front_left"
 		parent="front_axis_link"
-		steer_origin_xyz="0 ${track_width/2} 0"
-		steer_limit="${wheel_turn_limit}" />
+		suspension_origin_xyz="0 ${track_width/2} 0"
+		suspension_height="${suspension_height}"
+		steer_limit="${steer_limit}" />
 	<xacro:speed_wheel
 		prefix="rear_right"
 		parent="rear_axis_link"
-		origin_xyz="0 -${track_width/2} 0" />
+		suspension_origin_xyz="0 -${track_width/2} 0"
+		suspension_height="${suspension_height}" />
 	<xacro:speed_wheel
 		prefix="rear_left"
 		parent="rear_axis_link"
-		origin_xyz="0 ${track_width/2} 0" />
+		suspension_origin_xyz="0 ${track_width/2} 0"
+		suspension_height="${suspension_height}" />
     <gazebo>
         <plugin name="tigra_interface_plugin" filename="libackermann_raw_controller_plugin.so">

File: tigra_description/urdf/params.urdf.xacro (robot description, xacro)
@@ -4,9 +4,9 @@
     <xacro:property name="yaml_file" value="$(find tigra_description)/config/props.yaml" />
     <xacro:property name="props" value="${xacro.load_yaml(yaml_file)}" />
+    <!-- основные габариты -->
+    <xacro:property name="wheelbase" value="${props['wheelbase']}" />
+    <xacro:property name="track_width" value="${props['track_width']}" />
     <xacro:property name="front_wheel_2_front_bumper" value="0.3" />
     <xacro:property name="rear_wheel_2_rear_bumper" value="0.3" />
-    <xacro:property name="wheelbase" value="${props['wheelbase']}" />
-    <xacro:property name="track_width" value="${props['track_width']}" />
-    <!-- основные габариты -->
     <xacro:property name="body_length" value="${front_wheel_2_front_bumper+wheelbase+rear_wheel_2_rear_bumper}" />
     <xacro:property name="body_width" value="0.75" />
@@ -17,4 +17,6 @@
     <xacro:property name="wheel_radius" value="${props['wheel_radius']}" />
     <xacro:property name="wheel_mass" value="20" />
-    <xacro:property name="wheel_turn_limit" value="${pi/4}" />
+    <!-- характеристики подвески -->
+    <xacro:property name="steer_limit" value="${pi/4}" />
+    <xacro:property name="suspension_height" value="0.0" />
 </robot>

File: tigra_description/urdf/tigra_robocross21.urdf.xacro (robot description, xacro)
@@ -24,8 +24,8 @@
 		origin_xyz="-0.19 0.0 0.61"
 		origin_rpy="3.14159265 -0.01 3.14159265" />
-	<xacro:gps_sensor
-		prefix="front"
-		parent="base_footprint"
-		origin_xyz="0.0 0.0 ${body_heigth/2+0.1}"
+	<xacro:ublox_gps_sensor
+		prefix="top"
+		parent="base_link"
+		origin_xyz="0.0 0.0 ${body_heigth+0.1}"
 		origin_rpy="0.0 0.0 0.0" />
 	<!-- <xacro:elp_stereo
