Commit message: Added more params on plugin + urdf

File: spring_simple_sample/urdf/simple.urdf.xacro (robot description, xacro)
@@ -1,36 +1,36 @@
 <?xml version="1.0"?>
 <robot name="sample" xmlns:xacro="http://www.ros.org/wiki/xacro">
-	<property name="length" value="1.85" />
-	<property name="width" value="0.75" />
-	<property name="heigth" value="0.6" />
-	<property name="mass" value="420" />
-	<property name="wheel_width" value="0.25" />
-	<property name="wheel_radius" value="0.25" />
-	<property name="wheel_mass" value="20" />
-	<property name="wheel_turn_limit" value="${pi/4}" />
-	<property name="wheelbase" value="1.24" />
-	<property name="trackbase" value="1.00" />
-	<property name="base_center" value="${length/2}" />
+	<xacro:property name="length" value="1.85" />
+	<xacro:property name="width" value="0.75" />
+	<xacro:property name="heigth" value="0.6" />
+	<xacro:property name="mass" value="420" />
+	<xacro:property name="wheel_width" value="0.25" />
+	<xacro:property name="wheel_radius" value="0.25" />
+	<xacro:property name="wheel_mass" value="20" />
+	<xacro:property name="wheel_turn_limit" value="${pi/4}" />
+	<xacro:property name="wheelbase" value="1.24" />
+	<xacro:property name="trackbase" value="1.00" />
+	<xacro:property name="base_center" value="${length/2}" />
 	<!-- inertia -->
-	<macro name="null_inertial">
+	<xacro:macro name="null_inertial">
 		<inertial>
 			<mass value="0.001" />
 			<inertia ixx="0.001" ixy="0" ixz="0" iyy="0.001" iyz="0" izz="0.001" />
 		</inertial>
-	</macro>
-	<macro name="base_inertial" params="width length height mass *origin">
+	</xacro:macro>
+	<xacro:macro name="base_inertial" params="width length height mass *origin">
 		<inertial>
-			<insert_block name="origin" />
+			<xacro:insert_block name="origin" />
 			<mass value="${mass}" />
 			<inertia ixx="${mass * (width * width + height * height) / 12}" ixy="0" ixz="0" iyy="${mass * (length * length + height * height) / 12}" iyz="0" izz="${mass * (width * width + length * length) / 12}" />
 		</inertial>
-	</macro>
-	<macro name="wheel_inertial" params="r h mass *origin">
+	</xacro:macro>
+	<xacro:macro name="wheel_inertial" params="r h mass *origin">
 		<inertial>
-			<insert_block name="origin" />
+			<xacro:insert_block name="origin" />
 			<mass value="${mass}" />
 			<inertia ixx="${mass / 12 * (3 * r * r + h * h)}" ixy="0.0" ixz="0.0" iyy="${mass / 12 * (3 * r * r + h * h)}" iyz="0.0" izz="${mass / 2 * r * r}" />
 		</inertial>
-	</macro>
+	</xacro:macro>
 	<!-- xacro base new -->
 	<link name="base_link">

File: tigra_description/urdf/macros/camera.urdf.xacro (robot description, xacro)
@@ -1,8 +1,8 @@
 <?xml version="1.0"?>
 <robot xmlns:xacro="http://www.ros.org/wiki/xacro">
-	<property name="cam_mass" value="0" />
-	<property name="cam_size" value="0.02" />
+	<xacro:property name="cam_mass" value="0" />
+	<xacro:property name="cam_size" value="0.02" />
 	<xacro:include filename="$(find tigra_description)/urdf/macros/inertia.urdf.xacro" />
-	<macro name="camera_link" params="name direction position">
+	<xacro:macro name="camera_link" params="name direction position">
 		<link name="${direction}_${position}_cam_frame">
 			<visual>
@@ -20,6 +20,6 @@
 			<null_inertial />
 		</link>
-	</macro>
-	<macro name="single_camera" params="name direction position xyz rpy fov">
+	</xacro:macro>
+	<xacro:macro name="single_camera" params="name direction position xyz rpy fov">
 		<camera_link name="${name}" direction="${direction}" position="${position}" />
 		<joint name="${direction}_${position}_joint" type="fixed">
@@ -62,5 +62,5 @@
 					<alwaysOn>true</alwaysOn>
 					<updateRate>30.0</updateRate>
-					<cameraName>${robot_name}/${direction}/${position}</cameraName>
+					<cameraName>$(arg robot_name)/${direction}/${position}</cameraName>
 					<imageTopicName>image_raw</imageTopicName>
 					<frameName>${direction}_${position}_optical_frame</frameName>
@@ -74,4 +74,4 @@
 			</sensor>
 		</gazebo>
-	</macro>
+	</xacro:macro>
 </robot>

File: tigra_description/urdf/macros/damping_wheels.urdf.xacro (robot description, xacro)
@@ -1,11 +1,11 @@
 <?xml version="1.0"?>
 <robot xmlns:xacro="http://www.ros.org/wiki/xacro">
-	<property name="springStiffness" value="125000" />
-	<property name="springReference" value="0" />
+	<xacro:property name="springStiffness" value="125000" />
+	<xacro:property name="springReference" value="0" />
 	<xacro:include filename="$(find tigra_description)/urdf/macros/inertia.urdf.xacro" />
 	<xacro:include filename="$(find tigra_description)/urdf/macros/common.urdf.xacro" />
 	<xacro:include filename="$(find tigra_description)/urdf/macros/wheels.urdf.xacro" />
 	<!-- XACRO SPEED -->
-	<macro name="speed_wheel" params="name base_name xyz ">
+	<xacro:macro name="speed_wheel" params="name base_name xyz ">
 		<base_wheel name="wheel_${name}" />
 		<gazebo reference="${name}_spring_joint">
@@ -31,7 +31,7 @@
 			<limit effort="500.0" velocity="10.0" />
 		</joint>
-	</macro>
+	</xacro:macro>
 	<!-- XACRO STEER -->
-	<macro name="steer_wheel" params="name base_name xyz">
+	<xacro:macro name="steer_wheel" params="name base_name xyz">
 		<base_wheel name="wheel_${name}" />
 		<gazebo reference="${name}_spring_joint">
@@ -67,4 +67,4 @@
 			<limit effort="500" velocity="10.0" />
 		</joint>
-	</macro>
+	</xacro:macro>
 </robot>

File: tigra_description/urdf/macros/inertia.urdf.xacro (robot description, xacro)
@@ -9,5 +9,5 @@
 	<xacro:macro name="box_inertia" params="width length height mass *origin">
 		<inertial>
-			<insert_block name="origin" />
+			<xacro:insert_block name="origin" />
 			<mass value="${mass}" />
 			<inertia ixx="${mass * (width * width + height * height) / 12}" ixy="0" ixz="0" iyy="${mass * (length * length + height * height) / 12}" iyz="0" izz="${mass * (width * width + length * length) / 12}" />
@@ -16,5 +16,5 @@
 	<xacro:macro name="cylinder_inertia" params="r h mass *origin">
 		<inertial>
-			<insert_block name="origin" />
+			<xacro:insert_block name="origin" />
 			<mass value="${mass}" />
 			<inertia ixx="${mass / 12 * (3 * r * r + h * h)}" ixy="0.0" ixz="0.0" iyy="${mass / 12 * (3 * r * r + h * h)}" iyz="0.0" izz="${mass / 2 * r * r}" />

File: tigra_description/urdf/macros/tigra_params.urdf.xacro (robot description, xacro)
@@ -13,5 +13,6 @@
 	<xacro:property name="track_width" value="0.8" />
     <xacro:property name="lidar_location" value="${heigth/2+0.01}" />
-	<xacro:property name="robot_name" value="tigra" />
 	<xacro:property name="odom_frame" value="odom_wheel" />
+    <xacro:arg name="pub_tf" default="true" />
+    <xacro:arg name="robot_name" default="tigra" />
 </robot>

File: tigra_description/urdf/tigra.urdf.xacro (robot description, xacro)
@@ -31,14 +31,15 @@
 		<origin xyz="0 0 ${wheel_radius}" rpy="0 0 0" />
 	</joint>
-	<gazebo>
-		<plugin name="tigra_interface_plugin" filename="libtigra_interface_plugin.so">
-			<robotName>${robot_name}</robotName>
-			<maxSteerRad>${mid_wheel_turn_limit}</maxSteerRad>
-			<wheelbase>${wheelbase}</wheelbase>
-			<wheelRadius>${wheel_radius}</wheelRadius>
-			<trackWidth>${track_width}</trackWidth>
-			<odomFrame>${odom_frame}</odomFrame>
-		</plugin>
-	</gazebo>
+    <gazebo>
+        <plugin name="tigra_interface_plugin" filename="libtigra_interface_plugin.so">
+            <maxSteerRad>${mid_wheel_turn_limit}</maxSteerRad>
+            <wheelbase>${wheelbase}</wheelbase>
+            <wheelRadius>${wheel_radius}</wheelRadius>
+            <trackWidth>${track_width}</trackWidth>
+            <odomFrame>${odom_frame}</odomFrame>
+            <pubTf>$(arg pub_tf)</pubTf>
+            <robotName>$(arg robot_name)</robotName>
+        </plugin>
+    </gazebo>
 	<!-- steer_wheel -->
 	<xacro:steer_wheel name="joint_right_wheel_1" base_name="base_link" xyz="0.5 -0.375 -0.35" />

File: tigra_description/urdf/tigra_damping.urdf.xacro (robot description, xacro)
@@ -31,13 +31,15 @@
 		<origin xyz="0 0 ${wheel_radius}" rpy="0 0 0" />
 	</joint>
-	<gazebo>
-		<plugin name="tigra_interface_plugin" filename="libtigra_interface_plugin.so">
-			<robotName>${robot_name}</robotName>
-			<maxSteerRad>${mid_wheel_turn_limit}</maxSteerRad>
-			<wheelbase>${wheelbase}</wheelbase>
-			<wheelRadius>${wheel_radius}</wheelRadius>
-			<trackWidth>${track_width}</trackWidth>
-		</plugin>
-	</gazebo>
+    <gazebo>
+        <plugin name="tigra_interface_plugin" filename="libtigra_interface_plugin.so">
+            <maxSteerRad>${mid_wheel_turn_limit}</maxSteerRad>
+            <wheelbase>${wheelbase}</wheelbase>
+            <wheelRadius>${wheel_radius}</wheelRadius>
+            <trackWidth>${track_width}</trackWidth>
+            <odomFrame>${odom_frame}</odomFrame>
+            <pubTf>${arg pub_tf}</pubTf>
+            <robotName>${arg robot_name}</robotName>
+        </plugin>
+    </gazebo>
 	<!-- STEER WHEEL -->
 	<xacro:steer_wheel name="joint_right_wheel_1" base_name="base_link" xyz="0.5 -0.375 -0.35" />
