Commit message: #74 Added new plugin for full simulation of our system

File: tigra_description/urdf/macros/tigra_params.urdf.xacro (robot description, xacro)
@@ -1,17 +1,20 @@
 <?xml version="1.0"?>
 <robot xmlns:xacro="http://www.ros.org/wiki/xacro">
-    <xacro:property name="length" value="1.85" />
-    <xacro:property name="width" value="0.75" />
-    <xacro:property name="heigth" value="0.6" />
-    <xacro:property name="mass" value="420" />
+    <xacro:property name="yaml_file" value="$(find tigra_description)/config/props.yaml" />
+    <xacro:property name="props" value="${load_yaml(yaml_file)}" />
+    <xacro:property name="body_length" value="1.85" />
+    <xacro:property name="body_width" value="0.75" />
+    <xacro:property name="body_heigth" value="0.6" />
+    <xacro:property name="body_mass" value="340" />
     <xacro:property name="wheel_width" value="0.25" />
-    <xacro:property name="wheel_radius" value="0.25" />
+    <xacro:property name="wheel_radius" value="${props['wheel_radius']}" />
     <xacro:property name="wheel_mass" value="20" />
     <xacro:property name="wheel_turn_limit" value="${pi/4}" />
-	<xacro:property name="wheelbase" value="1.0" />
-	<xacro:property name="half_wheelbase" value="${wheelbase/2}" />
-	<xacro:property name="track_width" value="0.8" />
+    <xacro:property name="wheel_shift_pos" value="0.35" />
+    <xacro:property name="wheelbase" value="${props['wheelbase']}" />
+    <xacro:property name="half_wheelbase" value="${wheelbase/2}" />
+    <xacro:property name="track_width" value="${props['track_width']}" />
     <xacro:property name="lidar_location" value="${heigth/2+0.01}" />
-	<xacro:property name="odom_frame" value="odom_wheel" />
+    <xacro:property name="odom_frame" value="odom_wheel" />
     <xacro:arg name="pub_tf" default="true" />
     <xacro:arg name="robot_name" default="tigra" />

File: tigra_description/urdf/macros/wheels.urdf.xacro (robot description, xacro)
@@ -1,9 +1,9 @@
 <?xml version="1.0"?>
 <robot xmlns:xacro="http://www.ros.org/wiki/xacro">
-	<xacro:property name="wheel_width" value="0.25" />
-	<xacro:property name="wheel_radius" value="0.25" />
-	<xacro:property name="wheel_mass" value="20" />
+	<xacro:property name="wheel_effort" value="500" />
+	<xacro:property name="wheel_steer_effort" value="1000" />
+	<xacro:property name="wheel_velocity" value="10" />
 	<xacro:property name="wheel_turn_limit" value="${pi/4}" />
-	<xacro:property name="mid_wheel_turn_limit" value="${degrees_30}" />
+	<!-- <xacro:property name="mid_wheel_turn_limit" value="${degrees_30}" /> -->
 	<xacro:include filename="$(find tigra_description)/urdf/macros/inertia.urdf.xacro" />
 	<xacro:include filename="$(find tigra_description)/urdf/macros/common.urdf.xacro" />
@@ -23,12 +23,12 @@
 				</geometry>
 			</collision>
-			<cylinder_inertia r="${wheel_radius}" h="${wheel_width}" mass="${wheel_mass}">
+			<xacro:cylinder_inertia r="${wheel_radius}" h="${wheel_width}" mass="${wheel_mass}">
 				<origin xyz="0 0 0" rpy="${pi/2} 0 0" />
-			</cylinder_inertia>
+			</xacro:cylinder_inertia>
 		</link>
 	</xacro:macro>
 	<!-- XACRO SPEED -->
 	<xacro:macro name="speed_wheel" params="name base_name xyz ">
-		<base_wheel name="wheel_${name}" />
+		<xacro:base_wheel name="wheel_${name}" />
 		<joint name="${name}_speed_joint" type="continuous">
 			<parent link="${base_name}" />
@@ -36,12 +36,15 @@
 			<origin xyz="${xyz}" rpy="0 0 0" />
 			<axis xyz="0 1 0" />
-			<limit effort="500.0" velocity="10.0" />
+			<limit effort="${wheel_effort}" velocity="${wheel_velocity}" />
 		</joint>
 	</xacro:macro>
 	<!-- XACRO STEER -->
 	<xacro:macro name="steer_wheel" params="name base_name xyz">
-		<base_wheel name="wheel_${name}" />
+		<xacro:base_wheel name="wheel_${name}" />
+		<link name="steer_${name}">
+			<xacro:null_inertial />
+		</link>
 		<joint name="${name}_steer_joint" type="revolute">
-			<limit lower="${-wheel_turn_limit}" upper="${wheel_turn_limit}" effort="1000" velocity="0" />
+			<limit lower="${-wheel_turn_limit}" upper="${wheel_turn_limit}" effort="${wheel_steer_effort}" velocity="0" />
 			<parent link="${base_name}" />
 			<child link="steer_${name}" />
@@ -49,7 +52,4 @@
 			<axis xyz="0 0 1" />
 		</joint>
-		<link name="steer_${name}">
-			<null_inertial />
-		</link>
 		<joint name="${name}_speed_joint" type="continuous">
 			<parent link="steer_${name}" />
@@ -57,5 +57,5 @@
 			<origin xyz="0 0 0" rpy="0 0 0" />
 			<axis xyz="0 1 0" />
-			<limit effort="500" velocity="10.0" />
+			<limit effort="${wheel_effort}" velocity="${wheel_velocity}" />
 		</joint>
 	</xacro:macro>

File: tigra_description/urdf/tigra.urdf.xacro (robot description, xacro)
@@ -1,23 +1,21 @@
 <?xml version="1.0"?>
 <robot name="tigra" xmlns:xacro="http://www.ros.org/wiki/xacro">
+	<xacro:include filename="$(find tigra_description)/urdf/macros/tigra_params.urdf.xacro" />
 	<xacro:include filename="$(find tigra_description)/urdf/macros/wheels.urdf.xacro" />
 	<xacro:include filename="$(find tigra_description)/urdf/macros/inertia.urdf.xacro" />
-	<xacro:include filename="$(find tigra_description)/urdf/macros/tigra_params.urdf.xacro" />
-	<!-- xacro base new -->
 	<link name="base_link">
 		<visual>
 			<origin xyz="0 0 0" rpy="0 0 0" />
 			<geometry>
-				<box size="${length} ${width} ${heigth}" />
+				<box size="${body_length} ${body_width} ${body_heigth}" />
 			</geometry>
-			<material name="blue" />
 		</visual>
 		<collision name="base_collision">
 			<origin xyz="0 0 0" rpy="0 0 0" />
 			<geometry>
-				<box size="${length} ${width} ${heigth}" />
+				<box size="${body_length} ${body_width} ${body_heigth}" />
 			</geometry>
 		</collision>
-		<xacro:box_inertia width="${width}" length="${length}" height="${heigth}" mass="${mass}">
+		<xacro:box_inertia width="${body_width}" length="${body_length}" height="${body_heigth}" mass="${body_mass}">
 			<origin xyz="0 0 0" rpy="0 0 0" />
 		</xacro:box_inertia>
@@ -29,20 +27,20 @@
 		<parent link="base_footprint" />
 		<child link="base_link" />
-		<origin xyz="0 0 ${wheel_radius}" rpy="0 0 0" />
+		<origin xyz="0 0 ${wheel_radius+wheel_shift_pos}" rpy="0 0 0" />
 	</joint>
     <gazebo>
-        <plugin name="tigra_interface_plugin" filename="libackermann_controller_plugin.so">
-            <maxSteerRad>${mid_wheel_turn_limit}</maxSteerRad>
+        <plugin name="tigra_interface_plugin" filename="libackermann_raw_controller_plugin.so">
+            <!-- <maxSteerRad>${mid_wheel_turn_limit}</maxSteerRad> -->
             <wheelbase>${wheelbase}</wheelbase>
-            <wheelRadius>${wheel_radius}</wheelRadius>
+            <!-- <wheelRadius>${wheel_radius}</wheelRadius> -->
             <trackWidth>${track_width}</trackWidth>
-            <odomFrame>${odom_frame}</odomFrame>
-            <pubTf>$(arg pub_tf)</pubTf>
+            <!-- <odomFrame>${odom_frame}</odomFrame> -->
+            <!-- <pubTf>$(arg pub_tf)</pubTf> -->
             <robotName>$(arg robot_name)</robotName>
         </plugin>
     </gazebo>
-	<xacro:steer_wheel name="joint_right_wheel_1" base_name="base_link" xyz="0.5 -0.375 -0.35" />
-	<xacro:steer_wheel name="joint_left_wheel_1" base_name="base_link" xyz="0.5 0.375 -0.35" />
-	<xacro:speed_wheel name="joint_right_wheel_2" base_name="base_link" xyz="-0.5 -0.375 -0.35" />
-	<xacro:speed_wheel name="joint_left_wheel_2" base_name="base_link" xyz="-0.5 0.375 -0.35" />
+	<xacro:steer_wheel name="front_right_wheel" base_name="base_link" xyz="0.5 -0.375 -${wheel_shift_pos}" />
+	<xacro:steer_wheel name="front_left_wheel" base_name="base_link" xyz="0.5 0.375 -${wheel_shift_pos}" />
+	<xacro:speed_wheel name="rear_right_wheel" base_name="base_link" xyz="-0.5 -0.375 -${wheel_shift_pos}" />
+	<xacro:speed_wheel name="rear_left_wheel" base_name="base_link" xyz="-0.5 0.375 -${wheel_shift_pos}" />
 </robot>

File: tigra_description/urdf/tigra_damping.urdf.xacro (robot description, xacro)
@@ -9,15 +9,14 @@
 			<origin xyz="0 0 0" rpy="0 0 0" />
 			<geometry>
-				<box size="${length} ${width} ${heigth}" />
+				<box size="${body_length} ${body_width} ${body_heigth}" />
 			</geometry>
-			<material name="blue" />
 		</visual>
 		<collision name="base_collision">
 			<origin xyz="0 0 0" rpy="0 0 0" />
 			<geometry>
-				<box size="${length} ${width} ${heigth}" />
+				<box size="${body_length} ${body_width} ${body_heigth}" />
 			</geometry>
 		</collision>
-		<xacro:box_inertia width="${width}" length="${length}" height="${heigth}" mass="${mass}">
+		<xacro:box_inertia width="${body_width}" length="${body_length}" height="${body_heigth}" mass="${body_mass}">
 			<origin xyz="0 0 0" rpy="0 0 0" />
 		</xacro:box_inertia>
@@ -31,18 +30,18 @@
 		<origin xyz="0 0 ${wheel_radius}" rpy="0 0 0" />
 	</joint>
-    <gazebo>
-        <plugin name="tigra_interface_plugin" filename="libackermann_controller_plugin.so">
-            <maxSteerRad>${mid_wheel_turn_limit}</maxSteerRad>
-            <wheelbase>${wheelbase}</wheelbase>
-            <wheelRadius>${wheel_radius}</wheelRadius>
-            <trackWidth>${track_width}</trackWidth>
-            <odomFrame>${odom_frame}</odomFrame>
-            <pubTf>${arg pub_tf}</pubTf>
-            <robotName>${arg robot_name}</robotName>
-        </plugin>
-    </gazebo>
-	<xacro:steer_wheel name="joint_right_wheel_1" base_name="base_link" xyz="0.5 -0.375 -0.35" />
-	<xacro:steer_wheel name="joint_left_wheel_1" base_name="base_link" xyz="0.5 0.375 -0.35" />
-	<xacro:speed_wheel name="joint_right_wheel_2" base_name="base_link" xyz="-0.5 -0.375 -0.35" />
-	<xacro:speed_wheel name="joint_left_wheel_2" base_name="base_link" xyz="-0.5 0.375 -0.35" />
+	<gazebo>
+		<plugin name="tigra_interface_plugin" filename="libackermann_controller_plugin.so">
+			<maxSteerRad>${mid_wheel_turn_limit}</maxSteerRad>
+			<wheelbase>${wheelbase}</wheelbase>
+			<wheelRadius>${wheel_radius}</wheelRadius>
+			<trackWidth>${track_width}</trackWidth>
+			<odomFrame>${odom_frame}</odomFrame>
+			<pubTf>${arg pub_tf}</pubTf>
+			<robotName>${arg robot_name}</robotName>
+		</plugin>
+	</gazebo>
+	<xacro:steer_wheel name="front_right_wheel" base_name="base_link" xyz="0.5 -0.375 -0.35" />
+	<xacro:steer_wheel name="front_left_wheel" base_name="base_link" xyz="0.5 0.375 -0.35" />
+	<xacro:speed_wheel name="rear_right_wheel" base_name="base_link" xyz="-0.5 -0.375 -0.35" />
+	<xacro:speed_wheel name="rear_left_wheel" base_name="base_link" xyz="-0.5 0.375 -0.35" />
 </robot>

Commit message: #71 added IMU and GPS to model

File: tigra_description/urdf/macros/tigra_params.urdf.xacro (robot description, xacro)
@@ -11,9 +11,12 @@
     <xacro:property name="wheel_mass" value="20" />
     <xacro:property name="wheel_turn_limit" value="${pi/4}" />
-    <xacro:property name="wheel_shift_pos" value="0.35" />
+    <xacro:property name="wheel_shift_z" value="0.35" />
     <xacro:property name="wheelbase" value="${props['wheelbase']}" />
     <xacro:property name="half_wheelbase" value="${wheelbase/2}" />
     <xacro:property name="track_width" value="${props['track_width']}" />
     <xacro:property name="lidar_location" value="${heigth/2+0.01}" />
+    <xacro:property name="gps_height" value="0.05" />
+    <xacro:property name="imu_height" value="0.05" />
+    <xacro:property name="imu_length" value="0.2" />
     <xacro:property name="odom_frame" value="odom_wheel" />
     <xacro:arg name="pub_tf" default="true" />

File: tigra_description/urdf/tigra.urdf.xacro (robot description, xacro)
@@ -27,5 +27,5 @@
 		<parent link="base_footprint" />
 		<child link="base_link" />
-		<origin xyz="0 0 ${wheel_radius+wheel_shift_pos}" rpy="0 0 0" />
+		<origin xyz="0 0 ${wheel_radius+wheel_shift_z}" rpy="0 0 0" />
 	</joint>
     <gazebo>
@@ -40,7 +40,7 @@
         </plugin>
     </gazebo>
-	<xacro:steer_wheel name="front_right_wheel" base_name="base_link" xyz="0.5 -0.375 -${wheel_shift_pos}" />
-	<xacro:steer_wheel name="front_left_wheel" base_name="base_link" xyz="0.5 0.375 -${wheel_shift_pos}" />
-	<xacro:speed_wheel name="rear_right_wheel" base_name="base_link" xyz="-0.5 -0.375 -${wheel_shift_pos}" />
-	<xacro:speed_wheel name="rear_left_wheel" base_name="base_link" xyz="-0.5 0.375 -${wheel_shift_pos}" />
+	<xacro:steer_wheel name="front_right_wheel" base_name="base_link" xyz="${wheelbase/2} -${track_width/2} -${wheel_shift_z}" />
+	<xacro:steer_wheel name="front_left_wheel" base_name="base_link" xyz="${wheelbase/2} ${track_width/2} -${wheel_shift_z}" />
+	<xacro:speed_wheel name="rear_right_wheel" base_name="base_link" xyz="-${wheelbase/2} -${track_width/2} -${wheel_shift_z}" />
+	<xacro:speed_wheel name="rear_left_wheel" base_name="base_link" xyz="-${wheelbase/2} ${track_width/2} -${wheel_shift_z}" />
 </robot>

Commit message: fixed lidar_location

File: tigra_description/urdf/macros/tigra_params.urdf.xacro (robot description, xacro)
@@ -15,5 +15,5 @@
     <xacro:property name="half_wheelbase" value="${wheelbase/2}" />
     <xacro:property name="track_width" value="${props['track_width']}" />
-    <xacro:property name="lidar_location" value="${heigth/2+0.01}" />
+    <xacro:property name="lidar_location" value="${body_heigth/2+0.01}" />
     <xacro:property name="gps_height" value="0.05" />
     <xacro:property name="imu_height" value="0.05" />
